File: HW/shield_SDR_UN/proc.sch (KiCad schematic (older format))
At the start: 0 parts

Commit message: proc schematic done test.
Parts:
- added C? (x13): 100nF, Capacitor_SMD:C_0402_1005Metric, symbol pspice:C
- added C?: 4.7uF, Capacitor_SMD:C_1210_3225Metric, symbol pspice:C
- added C? (x2): 2.2uF, Capacitor_SMD:C_0402_1005Metric, symbol pspice:C
- added C? (x4): 1uF, Capacitor_SMD:C_0402_1005Metric, symbol pspice:C
- added U?: STM32F722ZETx, Package_QFP:LQFP-144_20x20mm_P0.5mm, symbol MCU_ST_STM32F7:STM32F722ZETx
Connections:
- net labels added: GND, JTCK-SWCLK, JTMS-SWDIO, VCC
- wire segments 0 -> 91
Other:
- note added: "PARA LOS PINES DE ALIMENTACION VDD / VSS\n"
- note added: "PARA VDDA/VSSA\n"
- note added: "pagina 100"
- note added: "pagina 100 y 157\n\n"
- note added: "para VDDSDMMC\n\n"
- note added: "para VDDUSB\nREVISAR\n\n\n"
- note added: "para VREF+\n"

Commit message: adicion potencia usb y osc procesador
Parts:
- removed C? (x13): 100nF, Capacitor_SMD:C_0402_1005Metric, symbol pspice:C
- removed C?: 4.7uF, Capacitor_SMD:C_1210_3225Metric, symbol pspice:C
- removed C? (x2): 2.2uF, Capacitor_SMD:C_0402_1005Metric, symbol pspice:C
- removed C? (x4): 1uF, Capacitor_SMD:C_0402_1005Metric, symbol pspice:C
- removed U?: STM32F722ZETx, Package_QFP:LQFP-144_20x20mm_P0.5mm, symbol MCU_ST_STM32F7:STM32F722ZETx
- added C? (x2): 10pF, symbol Device:C
- added C? (x2): 14pF, symbol Device:C
- added C? (x2): 2.2uF, Capacitor_SMD:C_0402_1005Metric, symbol Device:C
- added C? (x14): 100nF, Capacitor_SMD:C_0402_1005Metric, symbol Device:C
- added C? (x4): 1uF, Capacitor_SMD:C_0402_1005Metric, symbol Device:C
- added U?: STM32F722ZET, symbol shield_SDR_UN-rescue:STM32F722ZET
- added X?: GSG-XTAL4PIN, symbol hackrf-one-rescue:GSG-XTAL4PIN
- added X?: CRYSTAL, symbol hackrf-one-rescue:CRYSTAL
Connections:
- net labels added: 3v3 MCU, OSC32_IN, OSC32_OUT, OSC_IN, OSC_OUT, VDDA, VREF+
- net labels removed: JTCK-SWCLK, JTMS-SWDIO, VCC
- wire segments 91 -> 147
Other:
- note added: "ALTA FRECUENCIA\n"
- note added: "BAJA FRECUENCIA\n"
- note added: "C_L=(CL1*CL2)/(CL1+CL2)+CS\nC_L:capacitancia cristal\nCs:capacitancia cto entre 5 pf y 10pf\nCL1=CL2 typ (5pF-25pF)"
- note added: "R_EXT=1/(2*PI*frec*CL2)"
- note added: "recordar resistencia R_EXT\n"

Commit message: MAX2830 Symbol/Footprint created
Parts:
- X?: symbol hackrf-one-rescue:GSG-XTAL4PIN -> shield_SDR_UN-rescue:GSG-XTAL4PIN-hackrf-one-rescue
- X?: symbol hackrf-one-rescue:CRYSTAL -> shield_SDR_UN-rescue:CRYSTAL-hackrf-one-rescue
Changed lines of the file:
@@
 $EndComp
 $Comp
-L hackrf-one-rescue:GSG-XTAL4PIN X?
-U 0 0 5CD3D0E7
+L shield_SDR_UN-rescue:GSG-XTAL4PIN-hackrf-one-rescue X?
+U 1 1 5CD3D0E7
 P 2100 4700
 F 0 "X?" H 2100 5083 60  0000 C CNN
@@
 F 4 "25MHz - 10pF" H 2100 4879 50  0000 C CNN "frecuencia"
 F 5 "535-10297-1-ND////535-11296-1-ND" H 2100 4700 50  0001 C CNN "digikey"
-	0    2100 4700
+	1    2100 4700
 	1    0    0    -1
 $EndComp
@@
 $Comp
 L Device:C C?
-U 0 0 5CD67D93
+U 1 1 5CD67D93
 P 1450 4950
 F 0 "C?" H 1565 4996 50  0000 L CNN
@@
 F 2 "" H 1488 4800 50  0001 C CNN
 F 3 "~" H 1450 4950 50  0001 C CNN
-	0    1450 4950
-	1    0    0    -1
-$EndComp
-$Comp
-L Device:C C?
-U 0 0 5CD6880D
+	1    1450 4950
+	1    0    0    -1
+$EndComp
+$Comp
+L Device:C C?
+U 1 1 5CD6880D
 P 2750 4950
 F 0 "C?" H 2865 4996 50  0000 L CNN
@@
 F 2 "" H 2788 4800 50  0001 C CNN
 F 3 "~" H 2750 4950 50  0001 C CNN
-	0    2750 4950
+	1    2750 4950
 	1    0    0    -1
 $EndComp
@@
 $Comp
 L Device:C C?
-U 0 0 5CDDD934
+U 1 1 5CDDD934
 P 1400 6450
 F 0 "C?" H 1515 6496 50  0000 L CNN
@@
 F 2 "" H 1438 6300 50  0001 C CNN
 F 3 "~" H 1400 6450 50  0001 C CNN
-	0    1400 6450
-	1    0    0    -1
-$EndComp
-$Comp
-L Device:C C?
-U 0 0 5CDDD93E
+	1    1400 6450
+	1    0    0    -1
+$EndComp
+$Comp
+L Device:C C?
+U 1 1 5CDDD93E
 P 2700 6450
 F 0 "C?" H 2815 6496 50  0000 L CNN
@@
 F 2 "" H 2738 6300 50  0001 C CNN
 F 3 "~" H 2700 6450 50  0001 C CNN
-	0    2700 6450
+	1    2700 6450
 	1    0    0    -1
 $EndComp
@@
 recordar resistencia R_EXT\n
 $Comp
-L hackrf-one-rescue:CRYSTAL X?
-U 0 0 5CDEC498
+L shield_SDR_UN-rescue:CRYSTAL-hackrf-one-rescue X?
+U 1 1 5CDEC498
 P 2100 6200
 F 0 "X?" H 2100 6582 60  0000 C CNN
@@
 F 4 "32.768KHz -- 12pF" H 2100 6378 50  0000 C CNN "frecuencia"
 F 5 "SER4103CT-ND" H 2100 6200 50  0001 C CNN "digikey"
-	0    2100 6200
+	1    2100 6200
 	1    0    0    -1
 $EndComp
@@
 $Comp
 L Device:C C?
-U 0 0 5CE76675
+U 1 1 5CE76675
 P 1050 3350
 F 0 "C?" H 1050 3450 50  0000 L CNN
@@
 F 2 "Capacitor_SMD:C_0402_1005Metric" H 1088 3200 50  0001 C CNN
 F 3 "~" H 1050 3350 50  0001 C CNN
-	0    1050 3350
+	1    1050 3350
 	1    0    0    -1
 $EndComp
@@
 $Comp
 L Device:C C?
-U 0 0 5CE79C23
+U 1 1 5CE79C23
 P 2500 3450
 F 0 "C?" H 2500 3550 50  0000 L CNN
@@
 F 2 "Capacitor_SMD:C_0402_1005Metric" H 2538 3300 50  0001 C CNN
 F 3 "~" H 2500 3450 50  0001 C CNN
-	0    2500 3450
+	1    2500 3450
 	1    0    0    -1
 $EndComp
@@
 $Comp
 L Device:C C?
-U 0 0 5CE7B75E
+U 1 1 5CE7B75E
 P 2400 2200
 F 0 "C?" H 2400 2300 50  0000 L CNN
@@
 F 2 "Capacitor_SMD:C_0402_1005Metric" H 2438 2050 50  0001 C CNN
 F 3 "~" H 2400 2200 50  0001 C CNN
-	0    2400 2200
+	1    2400 2200
 	1    0    0    -1
 $EndComp
@@
 $Comp
 L Device:C C?
-U 0 0 5CE81CD3
+U 1 1 5CE81CD3
 P 1400 2200
 F 0 "C?" H 1400 2300 50  0000 L CNN
@@
 F 2 "Capacitor_SMD:C_0402_1005Metric" H 1438 2050 50  0001 C CNN
 F 3 "~" H 1400 2200 50  0001 C CNN
-	0    1400 2200
+	1    1400 2200
 	1    0    0    -1
 $EndComp
@@
 $Comp
 L Device:C C?
-U 0 0 5CE8BD3C
+U 1 1 5CE8BD3C
 P 1400 1200
 F 0 "C?" H 1400 1300 50  0000 L CNN
@@
 F 2 "Capacitor_SMD:C_0402_1005Metric" H 1438 1050 50  0001 C CNN
 F 3 "~" H 1400 1200 50  0001 C CNN
-	0    1400 1200
+	1    1400 1200
 	1    0    0    -1
 $EndComp
@@
 $Comp
 L Device:C C?
-U 0 0 5CE9042C
+U 1 1 5CE9042C
 P 1750 1200
 F 0 "C?" H 1750 1300 50  0000 L CNN
@@
 F 2 "Capacitor_SMD:C_0402_1005Metric" H 1788 1050 50  0001 C CNN
 F 3 "~" H 1750 1200 50  0001 C CNN
-	0    1750 1200
+	1    1750 1200
 	1    0    0    -1
 $EndComp
@@
 $Comp
 L Device:C C?
-U 0 0 5CE99526
+U 1 1 5CE99526
 P 2150 1200
 F 0 "C?" H 2150 1300 50  0000 L CNN
@@
 F 2 "Capacitor_SMD:C_0402_1005Metric" H 2188 1050 50  0001 C CNN
 F 3 "~" H 2150 1200 50  0001 C CNN
-	0    2150 1200
+	1    2150 1200
 	1    0    0    -1
 $EndComp
@@
 $Comp
 L Device:C C?
-U 0 0 5CE99531
+U 1 1 5CE99531
 P 2500 1200
 F 0 "C?" H 2500 1300 50  0000 L CNN
@@
 F 2 "Capacitor_SMD:C_0402_1005Metric" H 2538 1050 50  0001 C CNN
 F 3 "~" H 2500 1200 50  0001 C CNN
-	0    2500 1200
+	1    2500 1200
 	1    0    0    -1
 $EndComp
@@
 $Comp
 L Device:C C?
-U 0 0 5CE9B99A
+U 1 1 5CE9B99A
 P 2850 1200
 F 0 "C?" H 2850 1300 50  0000 L CNN
@@
 F 2 "Capacitor_SMD:C_0402_1005Metric" H 2888 1050 50  0001 C CNN
 F 3 "~" H 2850 1200 50  0001 C CNN
-	0    2850 1200
+	1    2850 1200
 	1    0    0    -1
 $EndComp
@@
 $Comp
 L Device:C C?
-U 0 0 5CE9B9A5
+U 1 1 5CE9B9A5
 P 3200 1200
 F 0 "C?" H 3200 1300 50  0000 L CNN
@@
 F 2 "Capacitor_SMD:C_0402_1005Metric" H 3238 1050 50  0001 C CNN
 F 3 "~" H 3200 1200 50  0001 C CNN
-	0    3200 1200
+	1    3200 1200
 	1    0    0    -1
 $EndComp
@@
 $Comp
 L Device:C C?
-U 0 0 5CE9E246
+U 1 1 5CE9E246
 P 3500 1200
 F 0 "C?" H 3500 1300 50  0000 L CNN
@@
 F 2 "Capacitor_SMD:C_0402_1005Metric" H 3538 1050 50  0001 C CNN
 F 3 "~" H 3500 1200 50  0001 C CNN
-	0    3500 1200
+	1    3500 1200
 	1    0    0    -1
 $EndComp
@@
 $Comp
 L Device:C C?
-U 0 0 5CE9E251
+U 1 1 5CE9E251
 P 3850 1200
 F 0 "C?" H 3850 1300 50  0000 L CNN
@@
 F 2 "Capacitor_SMD:C_0402_1005Metric" H 3888 1050 50  0001 C CNN
 F 3 "~" H 3850 1200 50  0001 C CNN
-	0    3850 1200
+	1    3850 1200
 	1    0    0    -1
 $EndComp
@@
 $Comp
 L Device:C C?
-U 0 0 5CEA1E50
+U 1 1 5CEA1E50
 P 4150 1200
 F 0 "C?" H 4150 1300 50  0000 L CNN
@@
 F 2 "Capacitor_SMD:C_0402_1005Metric" H 4188 1050 50  0001 C CNN
 F 3 "~" H 4150 1200 50  0001 C CNN
-	0    4150 1200
+	1    4150 1200
 	1    0    0    -1
 $EndComp
@@
 $Comp
 L Device:C C?
-U 0 0 5CEA1E5B
+U 1 1 5CEA1E5B
 P 4500 1200
 F 0 "C?" H 4500 1300 50  0000 L CNN
@@
 F 2 "Capacitor_SMD:C_0402_1005Metric" H 4538 1050 50  0001 C CNN
 F 3 "~" H 4500 1200 50  0001 C CNN
-	0    4500 1200
+	1    4500 1200
 	1    0    0    -1
 $EndComp
@@
 $Comp
 L Device:C C?
-U 0 0 5CEB7D81
+U 1 1 5CEB7D81
 P 1800 2200
 F 0 "C?" H 1800 2300 50  0000 L CNN
@@
 F 2 "Capacitor_SMD:C_0402_1005Metric" H 1838 2050 50  0001 C CNN
 F 3 "~" H 1800 2200 50  0001 C CNN
-	0    1800 2200
+	1    1800 2200
 	1    0    0    -1
 $EndComp
@@
 $Comp
 L Device:C C?
-U 0 0 5CEBA6A1
+U 1 1 5CEBA6A1
 P 2850 2200
 F 0 "C?" H 2850 2300 50  0000 L CNN
@@
 F 2 "Capacitor_SMD:C_0402_1005Metric" H 2888 2050 50  0001 C CNN
 F 3 "~" H 2850 2200 50  0001 C CNN
-	0    2850 2200
+	1    2850 2200
 	1    0    0    -1
 $EndComp
@@
 $Comp
 L Device:C C?
-U 0 0 5CEC20CF
+U 1 1 5CEC20CF
 P 1400 3350
 F 0 "C?" H 1400 3450 50  0000 L CNN
@@
 F 2 "Capacitor_SMD:C_0402_1005Metric" H 1438 3200 50  0001 C CNN
 F 3 "~" H 1400 3350 50  0001 C CNN
-	0    1400 3350
-	1    0    0    -1
-$EndComp
-$Comp
-L Device:C C?
-U 0 0 5CEC2843
+	1    1400 3350
+	1    0    0    -1
+$EndComp
+$Comp
+L Device:C C?
+U 1 1 5CEC2843
 P 2900 3450
 F 0 "C?" H 2900 3550 50  0000 L CNN
@@
 F 2 "Capacitor_SMD:C_0402_1005Metric" H 2938 3300 50  0001 C CNN
 F 3 "~" H 2900 3450 50  0001 C CNN
-	0    2900 3450
+	1    2900 3450
 	1    0    0    -1
 $EndComp
@@
 $Comp
 L Device:C C?
-U 0 0 5CE718F2
+U 1 1 5CE718F2
 P 5900 2400
 F 0 "C?" V 6000 2500 50  0000 L CNN
@@
 F 2 "Capacitor_SMD:C_0402_1005Metric" H 5938 2250 50  0001 C CNN
 F 3 "~" H 5900 2400 50  0001 C CNN
-	0    5900 2400
+	1    5900 2400
 	0    -1   -1   0
 $EndComp
 $Comp
 L Device:C C?
-U 0 0 5CEF657C
+U 1 1 5CEF657C
 P 5900 2700
 F 0 "C?" V 6000 2800 50  0000 L CNN
@@
 F 2 "Capacitor_SMD:C_0402_1005Metric" H 5938 2550 50  0001 C CNN
 F 3 "~" H 5900 2700 50  0001 C CNN
-	0    5900 2700
+	1    5900 2700
 	0    -1   -1   0
 $EndComp
@@
 Wire Wire Line
 	11100 900  11100 1050
+Connection ~ 1050 3100
+Connection ~ 2500 3200
+Connection ~ 2400 1950
+Connection ~ 1400 950
 $EndSCHEMATC

Commit message: STM32 connection updated
Parts:
- added BT?: Battery_Cell, symbol Device:Battery_Cell
- added C? (x2): 100nF, Capacitor_SMD:C_0402_1005Metric, symbol Device:C
- added D? (x2): LED, symbol Device:LED
- added J?: Conn_02x08_Top_Bottom, symbol Connector_Generic:Conn_02x08_Top_Bottom
- added R?: 10k, symbol Device:R
- added R?: 1K, symbol Device:R
- added R? (x2): 1.8k, symbol Device:R
- added R? (x15): 39, symbol Device:R
- added SW?: SW_Push, SWITCH_FSM1LPA, symbol FSM1LPTR:FSM1LPTR
- C? (x2): value 14pF -> 6pF
- C?: value 100nF -> 4.7uF
- X?: symbol shield_SDR_UN-rescue:GSG-XTAL4PIN-hackrf-one-rescue -> hackrf-one-rescue:GSG-XTAL4PIN; frecuencia 25MHz - 10pF -> 16MHz - 10pF
- X?: symbol shield_SDR_UN-rescue:CRYSTAL-hackrf-one-rescue -> hackrf-one-rescue:CRYSTAL; frecuencia 32.768KHz -- 12pF -> 32.768KHz -- 6pF
Connections:
- net 3v3 MCU: now also U?.143 (PDR_ON), U?.6 (VBAT), U?.95 (VDDUSB), BT?.1 (+), C?.1, R?.1
- net GND: now also BT?.2 (-), C?.2, C?.2, R?.2, R?.2, R?.2, SW?.3, SW?.4, SW?.5
- net CS_AD: now reaches U?.100 ((MCO1)(TIM1_CH1)(TIM8_BKIN2)(I2C3_SCL)(USART1_CK)(OTG_FS_SOF)(EVENTOUT)(PA8))
- net USART1_TX: now reaches U?.101 ((TIM1_CH2)(I2C3_SMBA)(SPI2_SCK/I2S2_CK)(USART1_TX)(EVENTOUT)(OTG_FS_VBUS)(PA9))
- net USART1_RX: now reaches U?.102 ((TIM1_CH3)(USART1_RX)(OTG_FS_ID)(EVENTOUT)(PA10))
- net JTAG0: now reaches U?.105 ((JTMS-SWDIO)(EVENTOUT)(PA13))
- net JTAG1: now reaches U?.109 ((JTCK-SWCLK)(EVENTOUT)(PA14))
- net JTAG2: now reaches U?.110 ((JTDI)(TIM2_CH1/TIM2_ETR)(SPI1_NSS/I2S1_WS)(SPI3_NSS/I2S3_WS)(UART4_RTS)(EVENTOUT)(PA15))
- net P_FPGA_1: now reaches U?.113 ((TRACED3)(SPI3_MOSI/I2S3_SD)(USART3_CK)(UART5_TX)(SDMMC1_CK)(EVENTOUT)(PC12))
- net P_FPGA_1: now also R?.1
- net P_FPGA_2: now reaches U?.114 ((CAN1_RX,_FMC_D2)(EVENTOUT)(PD0))
- net P_FPGA_2: now also R?.1
- net P_FPGA_3: now reaches U?.115 ((PD1)(CAN1_TX)(FMC_D3)(EVENTOUT))
- net P_FPGA_3: now also R?.1
- net P_FPGA_4: now reaches U?.116 ((TRACED2)(TIM3_ETR)(UART5_RX)(SDMMC1_CMD)(EVENTOUT)(PD2))
- net P_FPGA_4: now also R?.1
- net P_FPGA_5: now reaches U?.117 ((SPI2_SCK/I2S2_CK)(USART2_CTS)(FMC_CLK)(EVENTOUT)(PD3))
- net P_FPGA_5: now also R?.1
- net P_FPGA_6: now reaches U?.118 ((USART2_RTS)(FMC_NOE)(EVENTOUT)(PD4))
- net P_FPGA_6: now also R?.1
- net P_FPGA_7: now reaches U?.119 ((USART2_TX)(FMC_NWE)(EVENTOUT)(PD5))
- net P_FPGA_7: now also R?.1
- net P_FPGA_8: now reaches U?.122 ((SPI3_MOSI/I2S3_SD)(SAI1_SD_A)(USART2_RX)(SDMMC2_CK)(FMC_NWAIT)(EVENTOUT)(PD6))
- net P_FPGA_8: now also R?.1
- net P_FPGA_9: now reaches U?.123 ((USART2_CK_SDMMC2_CMD)(FMC_NE1)(EVENTOUT)(PD7))
- net P_FPGA_9: now also R?.1
- net P_FPGA_10: now reaches U?.124 ((USART6_RX)(QUADSPI_BK2_IO2)(SAI2_FS_B)(SDMMC2_D0)(FMC_NE2/FMC_NCE)(EVENTOUT)(PG9))
- net P_FPGA_10: now also R?.1
- net P_FPGA_11: now reaches U?.125 ((PG10)(SAI2_SD_B)(SDMMC2_D1)(FMC_NE3)(EVENTOUT))
- net P_FPGA_11: now also R?.1
- net P_FPGA_12: now reaches U?.126 ((PG11)(SDMMC2_D2)(FMC_INT)(EVENTOUT))
- net P_FPGA_12: now also R?.1
- net P_FPGA_13: now reaches U?.127 ((PG12)(LPTIM1_IN1)(USART6_RTS)(SDMMC2_D3)(FMC_NE4)(EVENTOUT))
- net P_FPGA_13: now also R?.1
- net P_FPGA_14: now reaches U?.128 ((PG13)(TRACED0)(LPTIM1_OUT)(USART6_CTS)(FMC_A24)(EVENTOUT))
- net P_FPGA_14: now also R?.1
- net P_FPGA_15: now reaches U?.129 ((PG14)(TRACED1)(LPTIM1_ETR)(USART6_TX)(QUADSPI_BK2_IO3)(FMC_A25)(EVENTOUT))
- net P_FPGA_15: now also R?.1
- net JTAG3: now reaches U?.133 ((JTDO/TRACESWO)(TIM2_CH2)(SPI1_SCK/I2S1_CK)(SPI3_SCK/I2S3_CK)(SDMMC2_D2)(EVENTOUT)(PB3))
- net JTAG4: now reaches U?.134 ((NJTRST)(TIM3_CH1)(SPI1_MISO,_SPI3_MISO)(SPI2_NSS/I2S2_WS)(SDMMC2_D3)(EVENTOUT)(PB4))
- net BOOT0: now reaches U?.138 (BOOT0)
- net BOOT0: now also R?.1
- net JTAG5: now reaches U?.25 (NRST)
- net JTAG5: now also C?.1, R?.2, SW?.1, SW?.2
- net XCVR_EN: now reaches U?.34 ((TIM2_CH1/TIM2_ETR)(TIM5_CH1)(TIM8_ETR)(USART2_CTS)(UART4_TX)(SAI2_SD_B)(EVENTOUT)(ADC1_IN0)(ADC2_IN0)(ADC3_IN0)(WKUP1)(PA0))
- net RSSI: now reaches U?.35 ((TIM2_CH2)(TIM5_CH2)(USART2_RTS)(UART4_RX)(QUADSPI_BK1_IO3)(SAI2_MCK_B)(EVENTOUT)(ADC1_IN1)(ADC2_IN1)(ADC3_IN1)(PA1))
- net TX_ENABLE: now reaches U?.36 ((TIM2_CH3)(TIM5_CH3)(TIM9_CH1)(USART2_TX)(SAI2_SCK_B)(EVENTOUT)(ADC1_IN2)(ADC2_IN2)(ADC3_IN2)(WKUP2)(PA2))
- net RX_ENABLE: now reaches U?.37 ((TIM2_CH4)(TIM5_CH4)(TIM9_CH2)(USART2_RX)(OTG_HS_ULPI_D0)(EVENTOUT)(ADC1_IN3)(ADC2_IN3)(ADC3_IN3)(PA3))
- net SPI1_NSS: now reaches U?.40 ((SPI1_NSS/I2S1_WS)(SPI3_NSS/I2S3_WS)(USART2_CK)_OTG_HS_SOF)(EVENTOUT)(ADC1_IN4)(ADC2_IN4)(DAC_OUT1)(PA4))
- net SPI1_SCK: now reaches U?.41 ((TIM2_CH1/TIM2_ETR)(TIM8_CH1N)(SPI1_SCK/I2S1_CK)(OTG_HS_ULPI_CK)(EVENTOUT)(ADC1_IN5)(ADC2_IN5)(DAC_OUT2)(PA5))
- net SPI1_MISO: now reaches U?.42 ((TIM1_BKIN)(TIM3_CH1)(TIM8_BKIN)(SPI1_MISO)(TIM13_CH1)(EVENTOUT)(ADC1_IN6)(ADC2_IN6)(PA6))
- net SPI1_MOSI: now reaches U?.43 ((TIM1_CH1N)(TIM3_CH2)(TIM8_CH1N)(SPI1_MOSI/I2S1_SD)(TIM14_CH1)(FMC_SDNWE)(EVENTOUT)(ADC1_IN7)(ADC2_IN7)(PA7))
- net !VAA_ENABLE: now reaches U?.46 ((TIM1_CH2N)(TIM3_CH3)(TIM8_CH2N)(UART4_CTS)(OTG_HS_ULPI_D1)(EVENTOUT)(ADC1_IN8)ADC2_IN8)(PB0))
- new net: D?.1 (K), R?.1 (x2)
- new net FPGA_B_1: R?.2
- new net FPGA_B_10: R?.2
- new net FPGA_B_11: R?.2
- new net FPGA_B_12: R?.2
- new net FPGA_B_13: R?.2
- new net FPGA_B_15: R?.2, R?.2
- new net FPGA_B_2: R?.2
- new net FPGA_B_3: R?.2
- new net FPGA_B_4: R?.2
- new net FPGA_B_5: R?.2
- new net FPGA_B_6: R?.2
- new net FPGA_B_7: R?.2
- new net FPGA_B_8: R?.2
- new net FPGA_B_9: R?.2
- new net LED1: D?.2 (A)
- new net LED2: D?.2 (A)
Other:
- note added: "REVISAR\n"
- moved on the sheet: C?, U?

Commit message: LED-PROC
Connections:
- net LED1: now also U?.56 ((PG0)(FMC_A10)(EVENTOUT))
- net LED2: now also U?.57 ((PG1)(FMC_A11)(EVENTOUT))
Changed lines of the file:
@@
 	1    0    0    -1
 $EndComp
+Wire Wire Line
+	6050 5550 5600 5550
+Wire Wire Line
+	6050 5650 5600 5650
+Text Label 5600 5550 0    50   ~ 0
+LED1
+Text Label 5600 5650 0    50   ~ 0
+LED2
 Wire Bus Line
 	7850 12700 7850 12900

Commit message: data bus proc-fpga
Parts:
- removed J?: Conn_02x08_Top_Bottom, symbol Connector_Generic:Conn_02x08_Top_Bottom
- added J?: Conn_02x10_Top_Bottom, symbol Connector_Generic:Conn_02x10_Top_Bottom
Connections:
- net GND: now also J?.10 (Pin_10), J?.20 (Pin_20)
- net GPIO_MCU_3: now reaches U?.1 ((PE2)(TRACECLK)(SPI4_SCK)(SAI1_MCLK_A)(QUADSPI_BK1_IO2)(FMC_A23)(EVENTOUT))
- net GPIO_MCU_3: now also J?.3 (Pin_3)
- net ADD_DAT_15: now reaches U?.10 ((PF0)(I2C2_SDA)(FMC_A0)(EVENTOUT))
- net ADD_DAT_16: now reaches U?.11 ((PF1)(I2C2_SCL)(FMC_A1)(EVENTOUT))
- net ADD_DAT_17: now reaches U?.12 ((PF2)(I2C2_SMBA)(FMC_A2)(EVENTOUT))
- net ADD_DAT_18: now reaches U?.13 ((PF3)(FMC_A3)(EVENTOUT)(ADC3_IN9))
- net ADD_DAT_19: now reaches U?.14 ((PF4)(FMC_A4)(EVENTOUT)(ADC3_IN14))
- net GPIO_MCU_1: now reaches U?.141 ((PE0)(TIM4_ETR)(LPTIM1_ETR)(UART8_Rx)(SAI2_MCK_A)(FMC_NBL0)(EVENTOUT))
- net GPIO_MCU_1: now also J?.1 (Pin_1)
- net GPIO_MCU_2: now reaches U?.142 ((PE1)(LPTIM1_IN2)(UART8_Tx)(FMC_NBL1)(EVENTOUT))
- net GPIO_MCU_2: now also J?.2 (Pin_2)
- net ADD_DAT_20: now reaches U?.15 ((PF5)(FMC_A5)(EVENTOUT)(ADC3_IN15))
- net ADD_DAT_21: now reaches U?.18 ((PF6)(TIM10_CH1)(SPI5_NSS)(SAI1_SD_B)(UART7_RX)(QUADSPI_BK1_IO3)(EVENTOUT)(ADC3_IN4))
- net ADD_DAT_22: now reaches U?.19 ((PF7)(TIM11_CH1)(SPI5_SCK)(SAI1_MCLK_B)(UART7_TX)(QUADSPI_BK1_IO2)(EVENTOUT)(ADC3_IN5))
- net GPIO_MCU_4: now reaches U?.2 ((PE3)(TRACED0)(SAI1_SD_B)(FMC_A19)(EVENTOUT))
- net GPIO_MCU_4: now also J?.4 (Pin_4)
- net ADD_DAT_23: now reaches U?.20 ((PF8)(SPI5_MISO)(SAI1_SCK_B)(UART7_RTS)(TIM13_CH1)(QUADSPI_BK1_IO0)(EVENTOUT)(ADC3_IN6))
- net ADD_DAT_24: now reaches U?.21 ((PF9)(SPI5_MOSI)(SAI1_FS_B)(UART7_CTS)(TIM14_CH1)(QUADSPI_BK1_IO1)(EVENTOUT)(ADC3_IN7))
- net ADD_DAT_25: now reaches U?.22 ((PF10)(EVENTOUT)(ADC3_IN8))
- net GPIO_MCU_5: now reaches U?.3 ((PE4)(TRACED1)(SPI4_NSS)(SAI1_FS_A)(FMC_A20)(EVENTOUT))
- net GPIO_MCU_5: now also J?.5 (Pin_5)
- net GPIO_MCU_6: now reaches U?.4 ((PE5)(TRACED2)(TIM9_CH1)(SPI4_MISO)(SAI1_SCK_A)(FMC_A21)(EVENTOUT))
- net GPIO_MCU_6: now also J?.6 (Pin_6)
- net ADD_DAT_26: now reaches U?.49 ((PF11)(SPI5_MOSI)(SAI2_SD_B)(FMC_SDNRAS)(EVENTOUT))
- net GPIO_MCU_7: now reaches U?.5 ((PE6)(TRACED3)(TIM1_BKIN2)(TIM9_CH2)(SPI4_MOSI)(SAI1_SD_A)(SAI2_MCK_B)(FMC_A22)(EVENTOUT))
- net GPIO_MCU_7: now also J?.7 (Pin_7)
- net ADD_DAT_27: now reaches U?.50 ((PF12)(FMC_A6)(EVENTOUT))
- net ADD_DAT_28: now reaches U?.53 ((PF13)(FMC_A7)(EVENTOUT))
- net ADD_DAT_29: now reaches U?.54 ((PF14)(FMC_A8)(EVENTOUT))
- net ADD_DAT_30: now reaches U?.55 ((PF15)(FMC_A9)(EVENTOUT))
- net GPIO_MCU_8: now reaches U?.58 ((PE7)(TIM1_ETR)(UART7_Rx)(QUADSPI_BK2_IO0)(FMC_D4)(EVENTOUT))
- net GPIO_MCU_8: now also J?.8 (Pin_8)
- net GPIO_MCU_9: now reaches U?.59 ((PE8)(TIM1_CH1N)(UART7_Tx)(QUADSPI_BK2_IO1)(FMC_D5)(EVENTOUT))
- net GPIO_MCU_9: now also J?.11 (Pin_11)
- net GPIO_MCU_10: now reaches U?.60 ((PE9)(TIM1_CH1)(UART7_RTS)(QUADSPI_BK2_IO2)(FMC_D6)(EVENTOUT))
- net GPIO_MCU_10: now also J?.12 (Pin_12)
- net GPIO_MCU_11: now reaches U?.63 ((PE10)(TIM1_CH2N)(UART7_CTS)(QUADSPI_BK2_IO3)(FMC_D7)(EVENTOUT))
- net GPIO_MCU_11: now also J?.13 (Pin_13)
- net GPIO_MCU_12: now reaches U?.64 ((PE11)(TIM1_CH2)(SPI4_NSS)(SAI2_SD_B)(FMC_D8)(EVENTOUT))
- net GPIO_MCU_12: now also J?.14 (Pin_14)
- net GPIO_MCU_13: now reaches U?.65 ((PE12)(TIM1_CH3N)(SPI4_SCK)(SAI2_SCK_B)(FMC_D9)(EVENTOUT))
- net GPIO_MCU_13: now also J?.15 (Pin_15)
- net GPIO_MCU_14: now reaches U?.66 ((PE13)(TIM1_CH3)(SPI4_MISO)(SAI2_FS_B)(FMC_D10)(EVENTOUT))
- net GPIO_MCU_14: now also J?.16 (Pin_16)
- net GPIO_MCU_15: now reaches U?.67 ((PE14)(TIM1_CH4)(SPI4_MOSI)(SAI2_MCK_B)(FMC_D11)(EVENTOUT))
- net GPIO_MCU_15: now also J?.17 (Pin_17)
- net GPIO_MCU_16: now reaches U?.68 ((PE15)(TIM1_BKIN)(FMC_D12)(EVENTOUT))
- net GPIO_MCU_16: now also J?.18 (Pin_18)
- net FPGA_B_1 renamed ADD_DAT_00
- net FPGA_B_10 renamed ADD_DAT_09
- net FPGA_B_11 renamed ADD_DAT_10
- net FPGA_B_12 renamed ADD_DAT_11
- net FPGA_B_13 renamed ADD_DAT_12
- net FPGA_B_15 renamed ADD_DAT_13
- net ADD_DAT_13: no longer R?.2
- net FPGA_B_2 renamed ADD_DAT_01
- net FPGA_B_3 renamed ADD_DAT_02
- net FPGA_B_4 renamed ADD_DAT_03
- net FPGA_B_5 renamed ADD_DAT_04
- net FPGA_B_6 renamed ADD_DAT_05
- net FPGA_B_7 renamed ADD_DAT_06
- net FPGA_B_8 renamed ADD_DAT_07
- net FPGA_B_9 renamed ADD_DAT_08
- new net +5V: J?.19 (Pin_19)
- new net 3V3 MCU: J?.9 (Pin_9)
- new net ADD_DAT_14: R?.2
