File: HW/shield_SDR_UN/proc.sch (KiCad schematic (older format))
At the start: 40 parts

Commit message: Footprints updated
Parts:
- removed C?: 10pF, Capacitor_SMD:C_0603_1608Metric_Pad1.05x0.95mm_HandSolder, symbol Device:C
- removed C?: 6pF, Capacitor_SMD:C_0603_1608Metric_Pad1.05x0.95mm_HandSolder, symbol Device:C
- removed C?: 2.2uF, Capacitor_SMD:C_0402_1005Metric, symbol Device:C
- removed D? (x2): LED, LED_SMD:LED_0805_2012Metric_Pad1.15x1.40mm_HandSolder, symbol Device:LED
- removed R? (x2): 1.8k, Resistor_SMD:R_0603_1608Metric_Pad1.05x0.95mm_HandSolder, symbol Device:R
- added C?: 2.2uF, Capacitor_SMD:C_0603_1608Metric_Pad1.05x0.95mm_HandSolder, symbol Device:C
- added C?: 10pF, Capacitor_SMD:C_0603_1608Metric_Pad1.05x0.95mm_HandSolder, symbol Device:C
- added C?: 6pF, Capacitor_SMD:C_0603_1608Metric_Pad1.05x0.95mm_HandSolder, symbol Device:C
- added D? (x2): LED, LED_SMD:LED_0805_2012Metric_Pad1.15x1.40mm_HandSolder, symbol Device:LED
- added R? (x2): 470, Resistor_SMD:R_0603_1608Metric_Pad1.05x0.95mm_HandSolder, symbol Device:R
- C?: Digikey (none) -> 1276-1027-1-ND
- C?: Digikey (none) -> 1276-2133-1-ND
- C?: footprint Capacitor_SMD:C_0402_1005Metric -> Capacitor_SMD:C_0603_1608Metric_Pad1.05x0.95mm_HandSolder; Digikey (none) -> 1276-1085-1-ND
- X?: Digikey (none) -> 644-1171-1-ND; digikey 644-1171-1-ND -> (none)
Connections:
- net GND: now also C?.1, C?.2, C?.2, D?.1 (K), D?.1 (K)
- net LED1: now also R?.1
- net LED2: now also R?.1
- net OSC32_OUT: now also C?.1
- net OSC_OUT: now also C?.1
- net at U?.106 (VCAP_2): now also C?.2
- new net: D?.2 (A), R?.2 (x2)
Other:
- note added: "Blue"
Changed lines of the file:
@@
 F 1 "10pF" H 1565 4905 50  0000 L CNN
 F 2 "Capacitor_SMD:C_0603_1608Metric_Pad1.05x0.95mm_HandSolder" H 1488 4800 50  0001 C CNN
-F 3 "~" H 1450 4950 50  0001 C CNN
+F 3 "http://www.samsungsem.com/kr/support/product-search/mlcc/__icsFiles/afieldfile/2016/12/01/Data%20sheet_CL10C100JB8NNNC.pdf" H 1450 4950 50  0001 C CNN
+F 4 "1276-1027-1-ND" H 1450 4950 50  0001 C CNN "Digikey"
 	1    1450 4950
-	1    0    0    -1
-$EndComp
-$Comp
-L Device:C C?
-U 1 1 5CD6880D
-P 2750 4950
-F 0 "C?" H 2865 4996 50  0000 L CNN
-F 1 "10pF" H 2865 4905 50  0000 L CNN
-F 2 "Capacitor_SMD:C_0603_1608Metric_Pad1.05x0.95mm_HandSolder" H 2788 4800 50  0001 C CNN
-F 3 "~" H 2750 4950 50  0001 C CNN
-	1    2750 4950
 	1    0    0    -1
 $EndComp
@@
 F 1 "6pF" H 1515 6405 50  0000 L CNN
 F 2 "Capacitor_SMD:C_0603_1608Metric_Pad1.05x0.95mm_HandSolder" H 1438 6300 50  0001 C CNN
-F 3 "~" H 1400 6450 50  0001 C CNN
+F 3 "www.samsungsem.com/kr/support/product-search/mlcc/CL10C060CB8NNNC.jsp" H 1400 6450 50  0001 C CNN
+F 4 "1276-2133-1-ND" H 1400 6450 50  0001 C CNN "Digikey"
 	1    1400 6450
-	1    0    0    -1
-$EndComp
-$Comp
-L Device:C C?
-U 1 1 5CDDD93E
-P 2700 6450
-F 0 "C?" H 2815 6496 50  0000 L CNN
-F 1 "6pF" H 2815 6405 50  0000 L CNN
-F 2 "Capacitor_SMD:C_0603_1608Metric_Pad1.05x0.95mm_HandSolder" H 2738 6300 50  0001 C CNN
-F 3 "~" H 2700 6450 50  0001 C CNN
-	1    2700 6450
 	1    0    0    -1
 $EndComp
@@
 F 3 "" H 2100 6200 60  0000 C CNN
 F 4 "32.768KHz -- 6pF" H 2100 6378 50  0000 C CNN "frecuencia"
-F 5 "644-1171-1-ND" H 2100 6200 50  0001 C CNN "digikey"
+F 5 "644-1171-1-ND" H 2100 6200 50  0001 C CNN "Digikey"
 	1    2100 6200
 	1    0    0    -1
@@
 U 1 1 5CE718F2
 P 5250 4250
-F 0 "C?" V 5350 4350 50  0000 L CNN
+F 0 "C?" V 5350 4300 50  0000 L CNN
 F 1 "2.2uF" V 5350 4000 50  0000 L CNN
-F 2 "Capacitor_SMD:C_0402_1005Metric" H 5288 4100 50  0001 C CNN
-F 3 "~" H 5250 4250 50  0001 C CNN
+F 2 "Capacitor_SMD:C_0603_1608Metric_Pad1.05x0.95mm_HandSolder" H 5288 4100 50  0001 C CNN
+F 3 "http://www.samsungsem.com/kr/support/product-search/mlcc/CL10A225KP8NNNC.jsp" H 5250 4250 50  0001 C CNN
+F 4 "1276-1085-1-ND" V 5250 4250 50  0001 C CNN "Digikey"
 	1    5250 4250
-	0    -1   -1   0
-$EndComp
-$Comp
-L Device:C C?
-U 1 1 5CEF657C
-P 5250 4550
-F 0 "C?" V 5350 4650 50  0000 L CNN
-F 1 "2.2uF" V 5350 4300 50  0000 L CNN
-F 2 "Capacitor_SMD:C_0402_1005Metric" H 5288 4400 50  0001 C CNN
-F 3 "~" H 5250 4550 50  0001 C CNN
-	1    5250 4550
 	0    -1   -1   0
 $EndComp
@@
 Text Notes 7550 1900 0    50   ~ 0
 REVISAR\n
-$Comp
-L Device:LED D?
-U 1 1 5CE7E335
-P 16550 2000
-F 0 "D?" V 16589 1883 50  0000 R CNN
-F 1 "LED" V 16498 1883 50  0000 R CNN
-F 2 "LED_SMD:LED_0805_2012Metric_Pad1.15x1.40mm_HandSolder" H 16550 2000 50  0001 C CNN
-F 3 "~" H 16550 2000 50  0001 C CNN
-	1    16550 2000
-	0    -1   -1   0
-$EndComp
-$Comp
-L Device:LED D?
-U 1 1 5CE83502
-P 17400 2000
-F 0 "D?" V 17439 1883 50  0000 R CNN
-F 1 "LED" V 17348 1883 50  0000 R CNN
-F 2 "LED_SMD:LED_0805_2012Metric_Pad1.15x1.40mm_HandSolder" H 17400 2000 50  0001 C CNN
-F 3 "~" H 17400 2000 50  0001 C CNN
-	1    17400 2000
-	0    -1   -1   0
-$EndComp
-$Comp
-L Device:R R?
-U 1 1 5CE8421C
-P 16550 2450
-F 0 "R?" H 16620 2496 50  0000 L CNN
-F 1 "1.8k" V 16550 2350 50  0000 L CNN
-F 2 "Resistor_SMD:R_0603_1608Metric_Pad1.05x0.95mm_HandSolder" V 16480 2450 50  0001 C CNN
-F 3 "~" H 16550 2450 50  0001 C CNN
-	1    16550 2450
-	1    0    0    -1
-$EndComp
-$Comp
-L Device:R R?
-U 1 1 5CE8472C
-P 17400 2450
-F 0 "R?" H 17470 2496 50  0000 L CNN
-F 1 "1.8k" V 17400 2350 50  0000 L CNN
-F 2 "Resistor_SMD:R_0603_1608Metric_Pad1.05x0.95mm_HandSolder" V 17330 2450 50  0001 C CNN
-F 3 "~" H 17400 2450 50  0001 C CNN
-	1    17400 2450
-	1    0    0    -1
-$EndComp
-$Comp
-L power:GND #PWR0174
-U 1 1 5CE8A343
-P 16550 2750
-F 0 "#PWR0174" H 16550 2500 50  0001 C CNN
-F 1 "GND" H 16555 2577 50  0000 C CNN
-F 2 "" H 16550 2750 50  0001 C CNN
-F 3 "" H 16550 2750 50  0001 C CNN
-	1    16550 2750
-	1    0    0    -1
-$EndComp
-$Comp
-L power:GND #PWR0175
-U 1 1 5CE906E0
-P 17400 2750
-F 0 "#PWR0175" H 17400 2500 50  0001 C CNN
-F 1 "GND" H 17405 2577 50  0000 C CNN
-F 2 "" H 17400 2750 50  0001 C CNN
-F 3 "" H 17400 2750 50  0001 C CNN
-	1    17400 2750
-	1    0    0    -1
-$EndComp
-Wire Wire Line
-	16550 1850 16100 1850
-Wire Wire Line
-	17400 1850 17000 1850
-Wire Wire Line
-	16550 2150 16550 2300
-Wire Wire Line
-	16550 2600 16550 2750
-Wire Wire Line
-	17400 2750 17400 2600
-Wire Wire Line
-	17400 2300 17400 2150
-Text Label 16100 1850 0    50   ~ 0
+Text Label 16550 1850 0    50   ~ 0
 LED1
 Text Label 17000 1850 0    50   ~ 0
@@
 	1    0    0    -1
 $EndComp
+$Comp
+L Device:LED D?
+U 1 1 5CEAA677
+P 16550 2650
+AR Path="/5CC082AD/5CEAA677" Ref="D?"  Part="1"
+AR Path="/5CFB52DC/5CEAA677" Ref="D?"  Part="1"
+F 0 "D?" V 16589 2533 50  0000 R CNN
+F 1 "LED" V 16498 2533 50  0000 R CNN
+F 2 "LED_SMD:LED_0805_2012Metric_Pad1.15x1.40mm_HandSolder" H 16550 2650 50  0001 C CNN
+F 3 "http://optoelectronics.liteon.com/upload/download/DS22-2000-239/LTST-S220TBKT.pdf" H 16550 2650 50  0001 C CNN
+F 4 "160-2032-1-ND" V 16550 2650 50  0001 C CNN "Digikey"
+	1    16550 2650
+	0    -1   -1   0
+$EndComp
+$Comp
+L power:GND #PWR?
+U 1 1 5CEAA678
+P 16550 2950
+F 0 "#PWR?" H 16550 2700 50  0001 C CNN
+F 1 "GND" H 16555 2777 50  0000 C CNN
+F 2 "" H 16550 2950 50  0001 C CNN
+F 3 "" H 16550 2950 50  0001 C CNN
+	1    16550 2950
+	1    0    0    -1
+$EndComp
+Wire Wire Line
+	16550 2350 16550 2500
+Wire Wire Line
+	16550 2800 16550 2950
+Text Notes 16400 2800 0    39   ~ 0
+Blue
+Wire Wire Line
+	16550 1850 16550 2050
+$Comp
+L Device:LED D?
+U 1 1 5CEAD127
+P 17000 2650
+AR Path="/5CC082AD/5CEAD127" Ref="D?"  Part="1"
+AR Path="/5CFB52DC/5CEAD127" Ref="D?"  Part="1"
+F 0 "D?" V 17039 2533 50  0000 R CNN
+F 1 "LED" V 16948 2533 50  0000 R CNN
+F 2 "LED_SMD:LED_0805_2012Metric_Pad1.15x1.40mm_HandSolder" H 17000 2650 50  0001 C CNN
+F 3 "http://optoelectronics.liteon.com/upload/download/DS22-2000-239/LTST-S220TBKT.pdf" H 17000 2650 50  0001 C CNN
+F 4 "160-2032-1-ND" V 17000 2650 50  0001 C CNN "Digikey"
+	1    17000 2650
+	0    -1   -1   0
+$EndComp
+$Comp
+L power:GND #PWR?
+U 1 1 5CEAD128
+P 17000 2950
+F 0 "#PWR?" H 17000 2700 50  0001 C CNN
+F 1 "GND" H 17005 2777 50  0000 C CNN
+F 2 "" H 17000 2950 50  0001 C CNN
+F 3 "" H 17000 2950 50  0001 C CNN
+	1    17000 2950
+	1    0    0    -1
+$EndComp
+Wire Wire Line
+	17000 2350 17000 2500
+Wire Wire Line
+	17000 2800 17000 2950
+Text Notes 16850 2800 0    39   ~ 0
+Blue
+Wire Wire Line
+	17000 1850 17000 2050
+$Comp
+L Device:R R?
+U 1 1 5CEC1673
+P 16550 2200
+F 0 "R?" H 16600 2250 50  0000 L CNN
+F 1 "470" V 16550 2100 50  0000 L CNN
+F 2 "Resistor_SMD:R_0603_1608Metric_Pad1.05x0.95mm_HandSolder" V 16480 2200 50  0001 C CNN
+F 3 "http://www.yageo.com/documents/recent/PYu-RC_Group_51_RoHS_L_10.pdf" H 16550 2200 50  0001 C CNN
+F 4 "311-470GRCT-ND" V 16550 2200 50  0001 C CNN "Digikey"
+	1    16550 2200
+	1    0    0    -1
+$EndComp
+$Comp
+L Device:R R?
+U 1 1 5CEC1B29
+P 17000 2200
+F 0 "R?" H 17050 2250 50  0000 L CNN
+F 1 "470" V 17000 2100 50  0000 L CNN
+F 2 "Resistor_SMD:R_0603_1608Metric_Pad1.05x0.95mm_HandSolder" V 16930 2200 50  0001 C CNN
+F 3 "http://www.yageo.com/documents/recent/PYu-RC_Group_51_RoHS_L_10.pdf" H 17000 2200 50  0001 C CNN
+F 4 "311-470GRCT-ND" V 17000 2200 50  0001 C CNN "Digikey"
+	1    17000 2200
+	1    0    0    -1
+$EndComp
+$Comp
+L Device:C C?
+U 1 1 5CE6AD58
+P 5250 4550
+F 0 "C?" V 5350 4600 50  0000 L CNN
+F 1 "2.2uF" V 5350 4300 50  0000 L CNN
+F 2 "Capacitor_SMD:C_0603_1608Metric_Pad1.05x0.95mm_HandSolder" H 5288 4400 50  0001 C CNN
+F 3 "http://www.samsungsem.com/kr/support/product-search/mlcc/CL10A225KP8NNNC.jsp" H 5250 4550 50  0001 C CNN
+F 4 "1276-1085-1-ND" V 5250 4550 50  0001 C CNN "Digikey"
+	1    5250 4550
+	0    -1   -1   0
+$EndComp
+$Comp
+L Device:C C?
+U 1 1 5CE7063F
+P 2750 4950
+F 0 "C?" H 2865 4996 50  0000 L CNN
+F 1 "10pF" H 2865 4905 50  0000 L CNN
+F 2 "Capacitor_SMD:C_0603_1608Metric_Pad1.05x0.95mm_HandSolder" H 2788 4800 50  0001 C CNN
+F 3 "http://www.samsungsem.com/kr/support/product-search/mlcc/__icsFiles/afieldfile/2016/12/01/Data%20sheet_CL10C100JB8NNNC.pdf" H 2750 4950 50  0001 C CNN
+F 4 "1276-1027-1-ND" H 2750 4950 50  0001 C CNN "Digikey"
+	1    2750 4950
+	1    0    0    -1
+$EndComp
+$Comp
+L Device:C C?
+U 1 1 5CE74AFC
+P 2700 6450
+F 0 "C?" H 2815 6496 50  0000 L CNN
+F 1 "6pF" H 2815 6405 50  0000 L CNN
+F 2 "Capacitor_SMD:C_0603_1608Metric_Pad1.05x0.95mm_HandSolder" H 2738 6300 50  0001 C CNN
+F 3 "www.samsungsem.com/kr/support/product-search/mlcc/CL10C060CB8NNNC.jsp" H 2700 6450 50  0001 C CNN
+F 4 "1276-2133-1-ND" H 2700 6450 50  0001 C CNN "Digikey"
+	1    2700 6450
+	1    0    0    -1
+$EndComp

Commit message: Footprints updated
Parts:
- R?: Digikey (none) -> 311-10KGRCT-ND
- R?: value 1K -> 1k; Digikey (none) -> 311-1.00KHRCT-ND
- X?: renamed from Y?e; symbol UL_ABM9G25000MHZB4YT:ABM8G-25.000MHZ-B4Y-T -> hackrf-one-rescue:GSG-XTAL4PIN
Changed lines of the file:
@@
-$EndComp
-$Comp
-L power:GND #PWR0164
-U 1 1 5CD657FB
-P 2050 4500
-F 0 "#PWR0164" H 2050 4250 50  0001 C CNN
-F 1 "GND" H 2055 4327 50  0000 C CNN
-F 2 "" H 2050 4500 50  0001 C CNN
-F 3 "" H 2050 4500 50  0001 C CNN
-	1    2050 4500
-	0    1    1    0
 $EndComp
 $Comp
 L power:GND #PWR0165
 U 1 1 5CD65D12
-P 2150 5000
-F 0 "#PWR0165" H 2150 4750 50  0001 C CNN
-F 1 "GND" H 2155 4827 50  0000 C CNN
-F 2 "" H 2150 5000 50  0001 C CNN
-F 3 "" H 2150 5000 50  0001 C CNN
-	1    2150 5000
-	1    0    0    -1
-$EndComp
-Wire Wire Line
-	2050 4500 2150 4500
-Wire Wire Line
-	2150 5000 2150 4900
+P 2050 5200
+F 0 "#PWR0165" H 2050 4950 50  0001 C CNN
+F 1 "GND" H 2055 5027 50  0000 C CNN
+F 2 "" H 2050 5200 50  0001 C CNN
+F 3 "" H 2050 5200 50  0001 C CNN
+	1    2050 5200
+	1    0    0    -1
+$EndComp
 $Comp
 L Device:C C?
@@
 Wire Wire Line
 	1450 4700 1100 4700
-Connection ~ 1450 4700
 Wire Wire Line
 	2750 4700 3150 4700
-Connection ~ 2750 4700
 Text Label 3150 6200 2    50   ~ 0
 OSC32_OUT
@@
 	1550 8000 1900 8000
 $Comp
-L Device:R R?
-U 1 1 5CD9E97E
-P 1900 8250
-F 0 "R?" H 1970 8296 50  0000 L CNN
-F 1 "1K" H 1970 8205 50  0000 L CNN
-F 2 "Resistor_SMD:R_0603_1608Metric_Pad1.05x0.95mm_HandSolder" V 1830 8250 50  0001 C CNN
-F 3 "~" H 1900 8250 50  0001 C CNN
-	1    1900 8250
-	1    0    0    -1
-$EndComp
-$Comp
 L power:GND #PWR0170
 U 1 1 5CD9F351
@@
 F 1 "10k" V 1350 9750 50  0000 L CNN
 F 2 "Resistor_SMD:R_0603_1608Metric_Pad1.05x0.95mm_HandSolder" V 1280 9800 50  0001 C CNN
-F 3 "~" H 1350 9800 50  0001 C CNN
+F 3 "http://www.yageo.com/documents/recent/PYu-RC_Group_51_RoHS_L_10.pdf" H 1350 9800 50  0001 C CNN
+F 4 "311-10KGRCT-ND" V 1350 9800 50  0001 C CNN "Digikey"
 	1    1350 9800
 	0    -1   -1   0
@@
 587-1897-1-ND
 $Comp
-L UL_ABM9G25000MHZB4YT:ABM8G-25.000MHZ-B4Y-T Y?e
+L hackrf-one-rescue:GSG-XTAL4PIN X?
 U 1 1 5D0A0635
-P 1950 4700
-F 0 "Y?e" H 2300 5050 60  0000 L CNN
-F 1 "GSG-XTAL4PIN" H 2300 4950 60  0000 L CNN
-F 2 "CRISTAL_4:GSG-XTAL3.2x2.5mm" H 2150 4340 60  0001 C CNN
-F 3 "" H 1950 4700 60  0000 C CNN
-F 4 "16MHz - 10pF" H 2600 4850 50  0000 C CNN "frecuencia"
-F 5 "535-10289-1-ND" H 1950 4700 50  0001 C CNN "digikey"
-	1    1950 4700
-	1    0    0    -1
-$EndComp
-Wire Wire Line
-	1450 4700 1950 4700
-Wire Wire Line
-	2350 4700 2750 4700
+P 2150 4700
+F 0 "X?" H 2250 5050 60  0000 L CNN
+F 1 "GSG-XTAL4PIN" H 2250 4950 60  0000 L CNN
+F 2 "CRISTAL_4:GSG-XTAL3.2x2.5mm" H 2350 4340 60  0001 C CNN
+F 3 "" H 2150 4700 60  0000 C CNN
+F 4 "16MHz - 10pF" H 2550 4850 50  0000 C CNN "frecuencia"
+F 5 "535-10289-1-ND" H 2150 4700 50  0001 C CNN "digikey"
+	1    2150 4700
+	1    0    0    -1
+$EndComp
 $Comp
 L Device:C C?
@@
 	1    0    0    -1
 $EndComp
+$Comp
+L power:GND #PWR?
+U 1 1 5CEA32F9
+P 2250 5200
+F 0 "#PWR?" H 2250 4950 50  0001 C CNN
+F 1 "GND" H 2255 5027 50  0000 C CNN
+F 2 "" H 2250 5200 50  0001 C CNN
+F 3 "" H 2250 5200 50  0001 C CNN
+	1    2250 5200
+	1    0    0    -1
+$EndComp
+Wire Wire Line
+	1850 4700 1450 4700
+Connection ~ 1450 4700
+Wire Wire Line
+	2450 4700 2750 4700
+Connection ~ 2750 4700
+Wire Wire Line
+	2250 5000 2250 5200
+Wire Wire Line
+	2050 5000 2050 5200
 Wire Bus Line
 	7850 12700 7850 12900
@@
 Wire Bus Line
 	11250 11550 11250 13150
+$Comp
+L Device:R R?
+U 1 1 5CD9E97E
+P 1900 8250
+F 0 "R?" H 1970 8296 50  0000 L CNN
+F 1 "1k" H 1970 8205 50  0000 L CNN
+F 2 "Resistor_SMD:R_0603_1608Metric_Pad1.05x0.95mm_HandSolder" V 1830 8250 50  0001 C CNN
+F 3 "http://www.yageo.com/documents/recent/PYu-RC_Group_51_RoHS_L_10.pdf" H 1900 8250 50  0001 C CNN
+F 4 " 311-1.00KHRCT-ND" H 1900 8250 50  0001 C CNN "Digikey"
+	1    1900 8250
+	1    0    0    -1
+$EndComp
 $EndSCHEMATC
