File: HW/shield_SDR_UN/proc.sch (KiCad schematic (older format))
At the start: 40 parts, among them J3 Conn_02x10_Top_Bottom, U5 STM32F722ZET, X3 CRYSTAL, X4 GSG-XTAL4PIN

Commit message: organizacion PCB
Parts:
- C103, C104, C90, C94: footprint Capacitor_SMD:C_0402_1005Metric -> Capacitor_SMD:C_0603_1608Metric_Pad1.05x0.95mm_HandSolder
Connections:
- net 3v3 MCU is gone; now on net 3V3 MCU: BT1.1 (+), C102.1, C103.1, C104.1, C105.1, C106.1, C107.1, C108.1, C109.1, C112.1, C87.1, C88.1, C90.1, C93.1, C95.1, C96.1, C97.1, C98.1, L1.1, R54.1, U5.108 (VDD), U5.121 (VDDSDMMC), U5.131 (VDD), U5.143 (PDR_ON), U5.144 (VDD), U5.17 (VDD), U5.30 (VDD), U5.32 (VREF+), U5.39 (VDD), U5.52 (VDD), U5.6 (VBAT), U5.62 (VDD), U5.72 (VDD), U5.84 (VDD), U5.95 (VDDUSB)
- no-connect marks 33 -> 34
Changed lines of the file:
@@
 Text Label 1700 1950 2    50   ~ 0
 VDDA
-Text GLabel 850  1950 0    50   Input ~ 0
-3v3 MCU
 Wire Wire Line
 	1000 1950 850  1950
-Text GLabel 2250 1950 0    50   Input ~ 0
-3v3 MCU
 Wire Wire Line
 	2400 1950 2250 1950
-Text GLabel 900  3100 0    50   Input ~ 0
-3v3 MCU
 Wire Wire Line
 	1050 3100 900  3100
-Text GLabel 2350 3200 0    50   Input ~ 0
-3v3 MCU
 Wire Wire Line
 	2500 3200 2350 3200
-Text GLabel 1250 950  0    50   Input ~ 0
-3v3 MCU
 Wire Wire Line
 	1400 950  1250 950
-Text GLabel 9600 2600 0    50   Input ~ 0
-3v3 MCU
 Wire Wire Line
 	9750 2600 9600 2600
 Wire Wire Line
 	9750 2600 9750 2800
-Text GLabel 10450 2750 1    50   Input ~ 0
-3v3 MCU
 Wire Wire Line
 	10450 2750 10450 2900
@@
 Connection ~ 2400 1950
 Connection ~ 1400 950
-Text GLabel 5650 3950 0    50   Input ~ 0
-3v3 MCU
 Wire Wire Line
 	6050 3950 5650 3950
@@
 	8800 2150 8050 2150
 Connection ~ 8050 2150
-Text GLabel 8100 2050 2    50   Input ~ 0
-3v3 MCU
 Wire Wire Line
 	8100 2050 8050 2050
@@
 Wire Wire Line
 	15350 5300 14950 5300
-Text GLabel 10550 2750 1    50   Input ~ 0
-3v3 MCU
 Wire Wire Line
 	10550 2750 10550 2900
@@
 F 0 "C104" H 2965 3546 50  0000 L CNN
 F 1 "1uF" H 2965 3355 50  0000 L CNN
-F 2 "Capacitor_SMD:C_0402_1005Metric" H 2938 3300 50  0001 C CNN
+F 2 "Capacitor_SMD:C_0603_1608Metric_Pad1.05x0.95mm_HandSolder" H 2938 3300 50  0001 C CNN
 F 3 "http://www.samsungsem.com/kr/support/product-search/mlcc/__icsFiles/afieldfile/2019/05/10/19-CL10A105KP8NNNC.pdf" H 2900 3450 50  0001 C CNN
 F 4 "1276-1182-1-ND" H 2900 3450 50  0001 C CNN "Digikey"
@@
 F 0 "C90" H 1465 3446 50  0000 L CNN
 F 1 "1uF" H 1465 3255 50  0000 L CNN
-F 2 "Capacitor_SMD:C_0402_1005Metric" H 1438 3200 50  0001 C CNN
+F 2 "Capacitor_SMD:C_0603_1608Metric_Pad1.05x0.95mm_HandSolder" H 1438 3200 50  0001 C CNN
 F 3 "http://www.samsungsem.com/kr/support/product-search/mlcc/__icsFiles/afieldfile/2019/05/10/19-CL10A105KP8NNNC.pdf" H 1400 3350 50  0001 C CNN
 F 4 "1276-1182-1-ND" H 1400 3350 50  0001 C CNN "Digikey"
@@
 F 0 "C94" H 1865 2296 50  0000 L CNN
 F 1 "1uF" H 1865 2105 50  0000 L CNN
-F 2 "Capacitor_SMD:C_0402_1005Metric" H 1838 2050 50  0001 C CNN
+F 2 "Capacitor_SMD:C_0603_1608Metric_Pad1.05x0.95mm_HandSolder" H 1838 2050 50  0001 C CNN
 F 3 "http://www.samsungsem.com/kr/support/product-search/mlcc/__icsFiles/afieldfile/2019/05/10/19-CL10A105KP8NNNC.pdf" H 1800 2200 50  0001 C CNN
 F 4 "1276-1182-1-ND" H 1800 2200 50  0001 C CNN "Digikey"
@@
 F 0 "C103" H 2915 2296 50  0000 L CNN
 F 1 "1uF" H 2915 2105 50  0000 L CNN
-F 2 "Capacitor_SMD:C_0402_1005Metric" H 2888 2050 50  0001 C CNN
+F 2 "Capacitor_SMD:C_0603_1608Metric_Pad1.05x0.95mm_HandSolder" H 2888 2050 50  0001 C CNN
 F 3 "http://www.samsungsem.com/kr/support/product-search/mlcc/__icsFiles/afieldfile/2019/05/10/19-CL10A105KP8NNNC.pdf" H 2850 2200 50  0001 C CNN
 F 4 "1276-1182-1-ND" H 2850 2200 50  0001 C CNN "Digikey"
@@
 Text GLabel 15350 6400 2    50   Input ~ 0
 I2C_SDA
-Text GLabel 1200 9750 0    50   Input ~ 0
-3v3 MCU
 $Comp
 L power:GND #PWR0110
@@
 	6050 13300 6500 13300
 NoConn ~ 14950 9100
+Text GLabel 8100 2050 2    50   Input ~ 0
+3V3 MCU
+Text GLabel 9600 2600 0    50   Input ~ 0
+3V3 MCU
+Text GLabel 10450 2750 1    50   Input ~ 0
+3V3 MCU
+Text GLabel 10550 2750 1    50   Input ~ 0
+3V3 MCU
+Text GLabel 850  1950 0    50   Input ~ 0
+3V3 MCU
+Text GLabel 2250 1950 0    50   Input ~ 0
+3V3 MCU
+Text GLabel 1250 950  0    50   Input ~ 0
+3V3 MCU
+Text GLabel 900  3100 0    50   Input ~ 0
+3V3 MCU
+Text GLabel 2350 3200 0    50   Input ~ 0
+3V3 MCU
+Text GLabel 1200 9750 0    50   Input ~ 0
+3V3 MCU
+Text GLabel 5650 3950 0    50   Input ~ 0
+3V3 MCU
+NoConn ~ 14950 6000
 $EndSCHEMATC

Commit message: Omega 2 PCB
Changed lines of the file:
@@
 Connection ~ 10150 2800
-Wire Wire Line
-	10150 2800 10050 2800
-Wire Wire Line
-	10050 2900 10050 2800
-Connection ~ 10050 2800
-Wire Wire Line
-	10050 2800 9950 2800
 Wire Wire Line
 	9950 2900 9950 2800
@@
 VREF+
 Text Label 10350 2700 3    50   ~ 0
-VDDA
-Wire Wire Line
-	10350 2900 10350 2700
-Text Label 1700 1950 2    50   ~ 0
 VDDA
 Wire Wire Line
@@
 3V3 MCU
 NoConn ~ 14950 6000
+Wire Wire Line
+	9950 2800 10050 2800
+Wire Wire Line
+	10050 2900 10050 2800
+Connection ~ 10050 2800
+Wire Wire Line
+	10050 2800 10150 2800
+Wire Wire Line
+	10350 2700 10350 2900
+Text Label 1800 1950 2    50   ~ 0
+VDDA
 $EndSCHEMATC
