File: HW/shield_SDR_UN/rf_front_end.sch (KiCad schematic (older format))
At the start: 80 parts, among them Q1 MOSFET_P, U1 MAX5864, U2 MAX2830

Commit message: Footprints updated
Parts:
- removed D1: LED, symbol Device:LED
- removed R?: 1.8k, Resistor_SMD:R_0603_1608Metric_Pad1.05x0.95mm_HandSolder, symbol Device:R
- added D?: LED, LED_SMD:LED_0805_2012Metric_Pad1.15x1.40mm_HandSolder, symbol Device:LED
- added R?: 470, Resistor_SMD:R_0603_1608Metric_Pad1.05x0.95mm_HandSolder, symbol Device:R
Other:
- note added: "Blue"
Changed lines of the file:
@@
-	0    -1   -1   0
-$EndComp
-$Comp
-L Device:LED D1
-U 1 1 5CE581D2
-P 1950 4250
-F 0 "D1" V 1989 4133 50  0000 R CNN
-F 1 "LED" V 1898 4133 50  0000 R CNN
-F 2 "" H 1950 4250 50  0001 C CNN
-F 3 "~" H 1950 4250 50  0001 C CNN
-	1    1950 4250
 	0    -1   -1   0
 $EndComp
@@
 $Comp
 L Device:R R?
-U 1 1 5CFC6C9A
+U 1 1 5CEDD000
 P 1700 4000
-F 0 "R?" V 1600 3900 50  0000 L CNN
-F 1 "1.8k" V 1700 3900 50  0000 L CNN
+F 0 "R?" V 1600 3950 50  0000 L CNN
+F 1 "470" V 1700 3900 50  0000 L CNN
 F 2 "Resistor_SMD:R_0603_1608Metric_Pad1.05x0.95mm_HandSolder" V 1630 4000 50  0001 C CNN
 F 3 "http://www.yageo.com/documents/recent/PYu-RC_Group_51_RoHS_L_10.pdf" H 1700 4000 50  0001 C CNN
-F 4 "311-1.8KGRTR-ND" V 1700 4000 50  0001 C CNN "Digikey"
+F 4 "311-470GRCT-ND" V 1700 4000 50  0001 C CNN "Digikey"
 	1    1700 4000
 	0    1    1    0
 $EndComp
+Text Notes 1800 4400 0    39   ~ 0
+Blue
+$Comp
+L Device:LED D?
+U 1 1 5CEDF6C9
+P 1950 4250
+AR Path="/5CC082AD/5CEDF6C9" Ref="D?"  Part="1"
+AR Path="/5CFB52DC/5CEDF6C9" Ref="D?"  Part="1"
+AR Path="/5CC081D2/5CEDF6C9" Ref="D?"  Part="1"
+F 0 "D?" V 1989 4133 50  0000 R CNN
+F 1 "LED" V 1898 4133 50  0000 R CNN
+F 2 "LED_SMD:LED_0805_2012Metric_Pad1.15x1.40mm_HandSolder" H 1950 4250 50  0001 C CNN
+F 3 "http://optoelectronics.liteon.com/upload/download/DS22-2000-239/LTST-S220TBKT.pdf" H 1950 4250 50  0001 C CNN
+F 4 "160-2032-1-ND" V 1950 4250 50  0001 C CNN "Digikey"
+	1    1950 4250
+	0    -1   -1   0
+$EndComp
 Wire Bus Line

Commit message: Footprints updated
Parts:
- removed R3, R4, R5: 1k, symbol Device:R
- added R? (x3): 1k, Resistor_SMD:R_0603_1608Metric_Pad1.05x0.95mm_HandSolder, symbol Device:R
- R6: footprint (none) -> Resistor_SMD:R_0603_1608Metric_Pad1.05x0.95mm_HandSolder; Digikey (none) -> 311-1.00KHRCT-ND
Changed lines of the file:
@@
 QD+
-$Comp
-L Device:R R6
-U 1 1 5CDD3BA8
-P 10950 2050
-F 0 "R6" V 10850 2050 50  0000 C CNN
-F 1 "1k" V 10950 2050 50  0000 C CNN
-F 2 "" V 10880 2050 50  0001 C CNN
-F 3 "~" H 10950 2050 50  0001 C CNN
-	1    10950 2050
-	0    -1   1    0
-$EndComp
 $Comp
 L Device:R R10
@@
 	11100 2050 11300 2050
 $Comp
-L Device:R R5
-U 1 1 5CDD2F9A
-P 10950 1800
-F 0 "R5" V 10850 1800 50  0000 C CNN
-F 1 "1k" V 10950 1800 50  0000 C CNN
-F 2 "" V 10880 1800 50  0001 C CNN
-F 3 "~" H 10950 1800 50  0001 C CNN
-	1    10950 1800
-	0    -1   1    0
-$EndComp
-$Comp
 L Device:R R9
 U 1 1 5CDD2F90
@@
 	11100 1800 11300 1800
 $Comp
-L Device:R R4
-U 1 1 5CDD2436
-P 10950 1550
-F 0 "R4" V 10850 1550 50  0000 C CNN
-F 1 "1k" V 10950 1550 50  0000 C CNN
-F 2 "" V 10880 1550 50  0001 C CNN
-F 3 "~" H 10950 1550 50  0001 C CNN
-	1    10950 1550
-	0    -1   1    0
-$EndComp
-$Comp
 L Device:R R8
 U 1 1 5CDD242C
@@
 Wire Wire Line
 	11100 1550 11300 1550
-$Comp
-L Device:R R3
-U 1 1 5CD943C7
-P 10950 1300
-F 0 "R3" V 10850 1300 50  0000 C CNN
-F 1 "1k" V 10950 1300 50  0000 C CNN
-F 2 "" V 10880 1300 50  0001 C CNN
-F 3 "~" H 10950 1300 50  0001 C CNN
-	1    10950 1300
-	0    -1   1    0
-$EndComp
 $Comp
 L Device:R R7
@@
 	0    -1   -1   0
 $EndComp
+$Comp
+L Device:R R6
+U 1 1 5CDD3BA8
+P 10950 2050
+F 0 "R6" V 10850 2050 50  0000 C CNN
+F 1 "1k" V 10950 2050 50  0000 C CNN
+F 2 "Resistor_SMD:R_0603_1608Metric_Pad1.05x0.95mm_HandSolder" V 10880 2050 50  0001 C CNN
+F 3 "http://www.yageo.com/documents/recent/PYu-RC_Group_51_RoHS_L_10.pdf" H 10950 2050 50  0001 C CNN
+F 4 " 311-1.00KHRCT-ND" V 10950 2050 50  0001 C CNN "Digikey"
+	1    10950 2050
+	0    -1   1    0
+$EndComp
+$Comp
+L Device:R R?
+U 1 1 5CE939F8
+P 10950 1800
+F 0 "R?" V 10850 1800 50  0000 C CNN
+F 1 "1k" V 10950 1800 50  0000 C CNN
+F 2 "Resistor_SMD:R_0603_1608Metric_Pad1.05x0.95mm_HandSolder" V 10880 1800 50  0001 C CNN
+F 3 "http://www.yageo.com/documents/recent/PYu-RC_Group_51_RoHS_L_10.pdf" H 10950 1800 50  0001 C CNN
+F 4 " 311-1.00KHRCT-ND" V 10950 1800 50  0001 C CNN "Digikey"
+	1    10950 1800
+	0    -1   1    0
+$EndComp
+$Comp
+L Device:R R?
+U 1 1 5CE94152
+P 10950 1550
+F 0 "R?" V 10850 1550 50  0000 C CNN
+F 1 "1k" V 10950 1550 50  0000 C CNN
+F 2 "Resistor_SMD:R_0603_1608Metric_Pad1.05x0.95mm_HandSolder" V 10880 1550 50  0001 C CNN
+F 3 "http://www.yageo.com/documents/recent/PYu-RC_Group_51_RoHS_L_10.pdf" H 10950 1550 50  0001 C CNN
+F 4 " 311-1.00KHRCT-ND" V 10950 1550 50  0001 C CNN "Digikey"
+	1    10950 1550
+	0    -1   1    0
+$EndComp
+$Comp
+L Device:R R?
+U 1 1 5CE94924
+P 10950 1300
+F 0 "R?" V 10850 1300 50  0000 C CNN
+F 1 "1k" V 10950 1300 50  0000 C CNN
+F 2 "Resistor_SMD:R_0603_1608Metric_Pad1.05x0.95mm_HandSolder" V 10880 1300 50  0001 C CNN
+F 3 "http://www.yageo.com/documents/recent/PYu-RC_Group_51_RoHS_L_10.pdf" H 10950 1300 50  0001 C CNN
+F 4 " 311-1.00KHRCT-ND" V 10950 1300 50  0001 C CNN "Digikey"
+	1    10950 1300
+	0    -1   1    0
+$EndComp
 Wire Bus Line

Commit message: OTRA VES FOOTPRINT
Parts:
- removed R1: 10k, symbol Device:R
- removed R10, R8, R9: 4.7k, symbol Device:R
- removed Y?e?: GSG-XTAL4PIN, CRISTAL_4:GSG-XTAL3.2x2.5mm, symbol UL_ABM9G25000MHZB4YT:ABM8G-25.000MHZ-B4Y-T
- added C?: 33pF, Capacitor_SMD:C_0603_1608Metric_Pad1.05x0.95mm_HandSolder, symbol Device:C
- added C?: 47pF, Capacitor_SMD:C_0603_1608Metric_Pad1.05x0.95mm_HandSolder, symbol Device:C
- added R?: 10k, Resistor_SMD:R_0603_1608Metric_Pad1.05x0.95mm_HandSolder, symbol Device:R
- added R? (x3): 4.7k, Resistor_SMD:R_0603_1608Metric_Pad1.05x0.95mm_HandSolder, symbol Device:R
- added X?: GSG-XTAL4PIN, CRISTAL_4:GSG-XTAL3.2x2.5mm, symbol hackrf-one-rescue:GSG-XTAL4PIN
- R7: footprint (none) -> Resistor_SMD:R_0603_1608Metric_Pad1.05x0.95mm_HandSolder; DESCRIPTION (none) -> 4.7 kOhms ±1% 0.1W, 1/10W; DIGIKEY (none) -> 311-4.70KHRCT-ND
Connections:
- net labels added: XTAL
- wire segments 354 -> 362
Changed lines of the file:
@@
 Wire Wire Line
 	1250 950  1250 1100
-$Comp
-L Device:R R1
-U 1 1 5CCE7B05
-P 1550 1100
-F 0 "R1" V 1450 1100 50  0000 C CNN
-F 1 "10k" V 1550 1100 50  0000 C CNN
-F 2 "" V 1480 1100 50  0001 C CNN
-F 3 "~" H 1550 1100 50  0001 C CNN
-	1    1550 1100
-	0    1    1    0
-$EndComp
 Wire Wire Line
 	1400 1100 1250 1100
@@
 Text Label 11300 1300 0    50   ~ 0
 QD+
-$Comp
-L Device:R R10
-U 1 1 5CDD3B9E
-P 10150 2050
-F 0 "R10" V 10050 2050 50  0000 C CNN
-F 1 "4.7k" V 10150 2050 50  0000 C CNN
-F 2 "" V 10080 2050 50  0001 C CNN
-F 3 "~" H 10150 2050 50  0001 C CNN
-	1    10150 2050
-	0    -1   1    0
-$EndComp
 Wire Wire Line
 	9850 2050 10000 2050
 Wire Wire Line
 	11100 2050 11300 2050
-$Comp
-L Device:R R9
-U 1 1 5CDD2F90
-P 10150 1800
-F 0 "R9" V 10050 1800 50  0000 C CNN
-F 1 "4.7k" V 10150 1800 50  0000 C CNN
-F 2 "" V 10080 1800 50  0001 C CNN
-F 3 "~" H 10150 1800 50  0001 C CNN
-	1    10150 1800
-	0    -1   1    0
-$EndComp
 Wire Wire Line
 	9850 1800 10000 1800
 Wire Wire Line
 	11100 1800 11300 1800
-$Comp
-L Device:R R8
-U 1 1 5CDD242C
-P 10150 1550
-F 0 "R8" V 10050 1550 50  0000 C CNN
-F 1 "4.7k" V 10150 1550 50  0000 C CNN
-F 2 "" V 10080 1550 50  0001 C CNN
-F 3 "~" H 10150 1550 50  0001 C CNN
-	1    10150 1550
-	0    -1   1    0
-$EndComp
 Wire Wire Line
 	9850 1550 10000 1550
@@
 $Comp
 L Device:R R7
-U 1 1 5CD95E2B
+U 0 0 5CD95E2B
 P 10150 1300
 F 0 "R7" V 10050 1300 50  0000 C CNN
 F 1 "4.7k" V 10150 1300 50  0000 C CNN
-F 2 "" V 10080 1300 50  0001 C CNN
+F 2 "Resistor_SMD:R_0603_1608Metric_Pad1.05x0.95mm_HandSolder" V 10080 1300 50  0001 C CNN
 F 3 "~" H 10150 1300 50  0001 C CNN
-	1    10150 1300
+F 4 "311-4.70KHRCT-ND" V 10150 1300 50  0001 C CNN "DIGIKEY"
+F 5 "4.7 kOhms ±1% 0.1W, 1/10W " V 10150 1300 50  0001 C CNN "DESCRIPTION"
+	0    10150 1300
 	0    -1   1    0
 $EndComp
@@
 L power:GND #PWR?
 U 1 1 5CEBA735
-P 8100 9450
+P 8100 10050
 AR Path="/5CC082AD/5CEBA735" Ref="#PWR?"  Part="1"
 AR Path="/5CC081D2/5CEBA735" Ref="#PWR?"  Part="1"
-F 0 "#PWR?" H 8100 9200 50  0001 C CNN
-F 1 "GND" H 8105 9277 50  0000 C CNN
-F 2 "" H 8100 9450 50  0001 C CNN
-F 3 "" H 8100 9450 50  0001 C CNN
-	1    8100 9450
-	0    1    1    0
+F 0 "#PWR?" H 8100 9800 50  0001 C CNN
+F 1 "GND" H 8105 9877 50  0000 C CNN
+F 2 "" H 8100 10050 50  0001 C CNN
+F 3 "" H 8100 10050 50  0001 C CNN
+	1    8100 10050
+	1    0    0    -1
 $EndComp
 $Comp
 L power:GND #PWR?
 U 1 1 5CEBA73D
-P 8200 9950
+P 8300 10050
 AR Path="/5CC082AD/5CEBA73D" Ref="#PWR?"  Part="1"
 AR Path="/5CC081D2/5CEBA73D" Ref="#PWR?"  Part="1"
-F 0 "#PWR?" H 8200 9700 50  0001 C CNN
-F 1 "GND" H 8205 9777 50  0000 C CNN
-F 2 "" H 8200 9950 50  0001 C CNN
-F 3 "" H 8200 9950 50  0001 C CNN
-	1    8200 9950
-	1    0    0    -1
-$EndComp
-Wire Wire Line
-	8100 9450 8200 9450
-Wire Wire Line
-	8200 9950 8200 9850
+F 0 "#PWR?" H 8300 9800 50  0001 C CNN
+F 1 "GND" H 8305 9877 50  0000 C CNN
+F 2 "" H 8300 10050 50  0001 C CNN
+F 3 "" H 8300 10050 50  0001 C CNN
+	1    8300 10050
+	1    0    0    -1
+$EndComp
+Wire Wire Line
+	8100 10050 8100 9950
 $Comp
 L Device:C C?
@@
 Wire Wire Line
 	7500 9650 7150 9650
-Connection ~ 7500 9650
 Wire Wire Line
 	8800 9650 9200 9650
-Connection ~ 8800 9650
-$Comp
-L UL_ABM9G25000MHZB4YT:ABM8G-25.000MHZ-B4Y-T Y?e?
-U 0 1 5CEBA77E
-P 8000 9650
-AR Path="/5CC082AD/5CEBA77E" Ref="Y?e?"  Part="1"
-AR Path="/5CC081D2/5CEBA77E" Ref="Y?e?"  Part="0"
-F 0 "Y?e?" H 8350 10000 60  0000 L CNN
-F 1 "GSG-XTAL4PIN" H 8350 9900 60  0000 L CNN
-F 2 "CRISTAL_4:GSG-XTAL3.2x2.5mm" H 8200 9290 60  0001 C CNN
-F 3 "" H 8000 9650 60  0000 C CNN
-F 4 "25MHz - 10pF" H 8650 9800 50  0000 C CNN "frecuencia"
-F 5 "535-13468-1-ND" H 8000 9650 50  0001 C CNN "digikey"
-F 6 "CRYSTAL 25.0000MHZ 10PF SMD" H 8000 9650 50  0001 C CNN "Descripcion"
-	0    8000 9650
-	1    0    0    -1
-$EndComp
-Wire Wire Line
-	7500 9650 8000 9650
-Wire Wire Line
-	8400 9650 8800 9650
 Text Label 9600 7950 0    50   ~ 0
 XA
@@
 	0    -1   1    0
 $EndComp
+$Comp
+L hackrf-one-rescue:GSG-XTAL4PIN X?
+U 0 1 5CE83378
+P 8200 9650
+AR Path="/5CC082AD/5CE83378" Ref="X?"  Part="1"
+AR Path="/5CC081D2/5CE83378" Ref="X?"  Part="0"
+F 0 "X?" H 8300 10000 60  0000 L CNN
+F 1 "GSG-XTAL4PIN" H 8300 9900 60  0000 L CNN
+F 2 "CRISTAL_4:GSG-XTAL3.2x2.5mm" H 8400 9290 60  0001 C CNN
+F 3 "" H 8200 9650 60  0000 C CNN
+F 4 "25MHz - 10pF" H 8600 9800 50  0000 C CNN "frecuencia"
+F 5 "535-13468-1-ND" H 8200 9650 50  0001 C CNN "digikey"
+F 6 "CRYSTAL 25.0000MHZ 10PF SMD" H 8200 9650 50  0001 C CNN "description"
+	0    8200 9650
+	1    0    0    -1
+$EndComp
+Wire Wire Line
+	8500 9650 8800 9650
+Connection ~ 8800 9650
+Wire Wire Line
+	7900 9650 7500 9650
+Connection ~ 7500 9650
+Wire Wire Line
+	8300 10050 8300 9950
+$Comp
+L Device:C C?
+U 0 0 5CEC998A
+P 11600 6600
+F 0 "C?" H 11715 6646 50  0000 L CNN
+F 1 "33pF" H 11715 6555 50  0000 L CNN
+F 2 "Capacitor_SMD:C_0603_1608Metric_Pad1.05x0.95mm_HandSolder" H 11638 6450 50  0001 C CNN
+F 3 "~" H 11600 6600 50  0001 C CNN
+	0    11600 6600
+	1    0    0    -1
+$EndComp
+$Comp
+L Device:C C?
+U 0 0 5CECB7A4
+P 11600 7100
+F 0 "C?" H 11715 7146 50  0000 L CNN
+F 1 "47pF" H 11715 7055 50  0000 L CNN
+F 2 "Capacitor_SMD:C_0603_1608Metric_Pad1.05x0.95mm_HandSolder" H 11638 6950 50  0001 C CNN
+F 3 "~" H 11600 7100 50  0001 C CNN
+	0    11600 7100
+	1    0    0    -1
+$EndComp
+$Comp
+L power:GND #PWR?
+U 1 1 5CEDA435
+P 11600 7400
+AR Path="/5CC082AD/5CEDA435" Ref="#PWR?"  Part="1"
+AR Path="/5CC081D2/5CEDA435" Ref="#PWR?"  Part="1"
+F 0 "#PWR?" H 11600 7150 50  0001 C CNN
+F 1 "GND" H 11605 7227 50  0000 C CNN
+F 2 "" H 11600 7400 50  0001 C CNN
+F 3 "" H 11600 7400 50  0001 C CNN
+	1    11600 7400
+	1    0    0    -1
+$EndComp
+Wire Wire Line
+	11600 7400 11600 7250
+Wire Wire Line
+	11600 6950 11600 6850
+Wire Wire Line
+	10750 7350 10750 6350
+Wire Wire Line
+	10750 6350 11600 6350
+Wire Wire Line
+	11600 6350 11600 6450
+Text Label 11950 6850 2    50   ~ 0
+XTAL
+Wire Wire Line
+	11950 6850 11600 6850
+Connection ~ 11600 6850
+Wire Wire Line
+	11600 6850 11600 6750
+Text Label 9200 4550 2    50   ~ 0
+XTAL
+Wire Wire Line
+	9200 4550 8850 4550
+$Comp
+L Device:R R?
+U 1 1 5CF8BBA1
+P 1550 1100
+AR Path="/5CC082AD/5CF8BBA1" Ref="R?"  Part="1"
+AR Path="/5CC081D2/5CF8BBA1" Ref="R?"  Part="1"
+F 0 "R?" V 1650 1100 50  0000 L CNN
+F 1 "10k" V 1550 1050 50  0000 L CNN
+F 2 "Resistor_SMD:R_0603_1608Metric_Pad1.05x0.95mm_HandSolder" V 1480 1100 50  0001 C CNN
+F 3 "http://www.yageo.com/documents/recent/PYu-RC_Group_51_RoHS_L_10.pdf" H 1550 1100 50  0001 C CNN
+F 4 "311-10KGRCT-ND" V 1550 1100 50  0001 C CNN "Digikey"
+	1    1550 1100
+	0    -1   -1   0
+$EndComp
+$Comp
+L Device:R R?
+U 0 0 5CFF1C5D
+P 10150 1550
+F 0 "R?" V 10050 1550 50  0000 C CNN
+F 1 "4.7k" V 10150 1550 50  0000 C CNN
+F 2 "Resistor_SMD:R_0603_1608Metric_Pad1.05x0.95mm_HandSolder" V 10080 1550 50  0001 C CNN
+F 3 "~" H 10150 1550 50  0001 C CNN
+F 4 "311-4.70KHRCT-ND" V 10150 1550 50  0001 C CNN "DIGIKEY"
+F 5 "4.7 kOhms ±1% 0.1W, 1/10W " V 10150 1550 50  0001 C CNN "DESCRIPTION"
+	0    10150 1550
+	0    -1   1    0
+$EndComp
+$Comp
+L Device:R R?
+U 0 0 5CFF22BF
+P 10150 1800
+F 0 "R?" V 10050 1800 50  0000 C CNN
+F 1 "4.7k" V 10150 1800 50  0000 C CNN
+F 2 "Resistor_SMD:R_0603_1608Metric_Pad1.05x0.95mm_HandSolder" V 10080 1800 50  0001 C CNN
+F 3 "~" H 10150 1800 50  0001 C CNN
+F 4 "311-4.70KHRCT-ND" V 10150 1800 50  0001 C CNN "DIGIKEY"
+F 5 "4.7 kOhms ±1% 0.1W, 1/10W " V 10150 1800 50  0001 C CNN "DESCRIPTION"
+	0    10150 1800
+	0    -1   1    0
+$EndComp
+$Comp
+L Device:R R?
+U 0 0 5CFF295F
+P 10150 2050
+F 0 "R?" V 10050 2050 50  0000 C CNN
+F 1 "4.7k" V 10150 2050 50  0000 C CNN
+F 2 "Resistor_SMD:R_0603_1608Metric_Pad1.05x0.95mm_HandSolder" V 10080 2050 50  0001 C CNN
+F 3 "~" H 10150 2050 50  0001 C CNN
+F 4 "311-4.70KHRCT-ND" V 10150 2050 50  0001 C CNN "DIGIKEY"
+F 5 "4.7 kOhms ±1% 0.1W, 1/10W " V 10150 2050 50  0001 C CNN "DESCRIPTION"
+	0    10150 2050
+	0    -1   1    0
+$EndComp

Commit message: OTRA VES FOOTPRINT_v1
Changed lines of the file:
@@
 $Comp
 L Device:R R7
-U 0 0 5CD95E2B
+U 1 1 5CD95E2B
 P 10150 1300
 F 0 "R7" V 10050 1300 50  0000 C CNN
@@
 F 4 "311-4.70KHRCT-ND" V 10150 1300 50  0001 C CNN "DIGIKEY"
 F 5 "4.7 kOhms ±1% 0.1W, 1/10W " V 10150 1300 50  0001 C CNN "DESCRIPTION"
-	0    10150 1300
+	1    10150 1300
 	0    -1   1    0
 $EndComp
@@
 $Comp
 L Device:C C?
-U 0 0 5CEC998A
+U 1 1 5CEC998A
 P 11600 6600
 F 0 "C?" H 11715 6646 50  0000 L CNN
@@
 F 2 "Capacitor_SMD:C_0603_1608Metric_Pad1.05x0.95mm_HandSolder" H 11638 6450 50  0001 C CNN
 F 3 "~" H 11600 6600 50  0001 C CNN
-	0    11600 6600
-	1    0    0    -1
-$EndComp
-$Comp
-L Device:C C?
-U 0 0 5CECB7A4
+	1    11600 6600
+	1    0    0    -1
+$EndComp
+$Comp
+L Device:C C?
+U 1 1 5CECB7A4
 P 11600 7100
 F 0 "C?" H 11715 7146 50  0000 L CNN
@@
 F 2 "Capacitor_SMD:C_0603_1608Metric_Pad1.05x0.95mm_HandSolder" H 11638 6950 50  0001 C CNN
 F 3 "~" H 11600 7100 50  0001 C CNN
-	0    11600 7100
+	1    11600 7100
 	1    0    0    -1
 $EndComp
@@
 $Comp
 L Device:R R?
-U 0 0 5CFF1C5D
+U 1 1 5CFF1C5D
 P 10150 1550
 F 0 "R?" V 10050 1550 50  0000 C CNN
@@
 F 4 "311-4.70KHRCT-ND" V 10150 1550 50  0001 C CNN "DIGIKEY"
 F 5 "4.7 kOhms ±1% 0.1W, 1/10W " V 10150 1550 50  0001 C CNN "DESCRIPTION"
-	0    10150 1550
+	1    10150 1550
 	0    -1   1    0
 $EndComp
 $Comp
 L Device:R R?
-U 0 0 5CFF22BF
+U 1 1 5CFF22BF
 P 10150 1800
 F 0 "R?" V 10050 1800 50  0000 C CNN
@@
 F 4 "311-4.70KHRCT-ND" V 10150 1800 50  0001 C CNN "DIGIKEY"
 F 5 "4.7 kOhms ±1% 0.1W, 1/10W " V 10150 1800 50  0001 C CNN "DESCRIPTION"
-	0    10150 1800
+	1    10150 1800
 	0    -1   1    0
 $EndComp
 $Comp
 L Device:R R?
-U 0 0 5CFF295F
+U 1 1 5CFF295F
 P 10150 2050
 F 0 "R?" V 10050 2050 50  0000 C CNN
@@
 F 4 "311-4.70KHRCT-ND" V 10150 2050 50  0001 C CNN "DIGIKEY"
 F 5 "4.7 kOhms ±1% 0.1W, 1/10W " V 10150 2050 50  0001 C CNN "DESCRIPTION"
-	0    10150 2050
+	1    10150 2050
 	0    -1   1    0
 $EndComp

Commit message: RF-Front-end connections
Parts:
- removed C?: 100nF, Capacitor_SMD:C_0603_1608Metric_Pad1.05x0.95mm_HandSolder, symbol Device:C
- removed C?: 1.8pF, Capacitor_SMD:C_0603_1608Metric_Pad1.05x0.95mm_HandSolder, symbol Device:C
- added C? (x2): 100nF, Capacitor_SMD:C_0603_1608Metric_Pad1.05x0.95mm_HandSolder, symbol Device:C
- added C?: 100pF, Capacitor_SMD:C_0603_1608Metric_Pad1.05x0.95mm_HandSolder, symbol Device:C
- added C?: 2.2nF, Capacitor_SMD:C_0603_1608Metric_Pad1.05x0.95mm_HandSolder, symbol Device:C
- added C?: 68pF, Capacitor_SMD:C_0603_1608Metric_Pad1.05x0.95mm_HandSolder, symbol Device:C
- added C?: 1.8pF, Capacitor_SMD:C_0603_1608Metric_Pad1.05x0.95mm_HandSolder, symbol Device:C
- added R?: 1.2k, Resistor_SMD:R_0603_1608Metric_Pad1.05x0.95mm_HandSolder, symbol Device:R
- added R?: 750, Resistor_SMD:R_0603_1608Metric_Pad1.05x0.95mm_HandSolder, symbol Device:R
- C?: Digikey (none) -> 1276-2218-1-ND
- C?: Digikey (none) -> 1276-1070-1-ND
- C?: Digikey (none) -> 1276-1037-1-ND
- U1: footprint (none) -> lib:MAX5864ETM&plus_; Digikey (none) -> MAX5864ETM+-ND
- U2: Digikey (none) -> MAX2830ETM+TCT-ND
- X?: Digikey (none) -> 535-13468-1-ND; digikey 535-13468-1-ND -> (none)
Connections:
- net labels added: rf_!SHDN, rf_ANTSEL, rf_RXTX, rf_TUNE
- net labels removed: rfB1, rfB2, rfB3, rfB4, rfB5, rfB6, rfB7
- wire segments 362 -> 374
- no-connect marks 5 -> 13

Commit message: OTRA VES FOOTPRINT_v2
Parts:
- removed R? (x2): 39, Resistor_SMD:R_0402_1005Metric, symbol Device:R
- added C? (x4): 100nF, Capacitor_SMD:C_0603_1608Metric_Pad1.05x0.95mm_HandSolder, symbol Device:C
- added R? (x2): 39, Resistor_SMD:R_0603_1608Metric_Pad1.05x0.95mm_HandSolder, symbol Device:R
- R?: footprint Resistor_SMD:R_0402_1005Metric -> Resistor_SMD:R_0603_1608Metric_Pad1.05x0.95mm_HandSolder; descripcion RES 39 OHM 1/16W 5% 0402 SMD -> RES SMD 39 OHM 1% 1/10W 0603; digikey RMCF0402JT39R0CT-ND -> 311-39.0HRCT-ND; part numer RMCF0402JT39R0 -> RC0603FR-0739RL
Connections:
- net labels added: CS_AD, PROC-MAX2837 [0:7], PROC-MAX5864 [0:2], RSSI, RX_ENABLE, SPI1_MISO, SPI1_MOSI, SPI1_NSS, SPI1_SCK, TX_ENABLE, XCVR_EN
- wire segments 374 -> 408
Other:
- note added: "OJO CON ESTOS PINES LOS COLOQUE \nCOMO EL HACK COMUNICACION CON EL MICRO"
- note added: "decoupling capacitor per power supply pin \nSI5351C"
- moved on the sheet: C?
