File: HW/shield_SDR_UN/FPGA.sch (KiCad schematic (older format))
At the start: 71 parts, among them J1 Conn_02x09_Odd_Even, J2 Conn_02x08_Odd_Even, U4 XC6SLX9-2TQG144C, X2 ASE-xxxMHz

Commit message: organizacion PCB
Connections:
- net I2C_SDA: now also J2.13 (Pin_13)
Other:
- moved on the sheet: J2, R40, R41, R42, R43, R44, R45, R46, R47, R48

Commit message: organizacion PCB_V2
Parts:
- added C127, C129, C130, C131, C132, C133, C135, C136, C137, C141, C142, C146, C147, C148, C149: 47nF, Capacitor_SMD:C_0603_1608Metric_Pad1.05x0.95mm_HandSolder, symbol Device:C
- added C128, C138, C139, C140, C150, C151: 0.47uF, Capacitor_SMD:C_0603_1608Metric_Pad1.05x0.95mm_HandSolder, symbol Device:C
- added C134, C143, C144, C145, C152: 4.7uF, Capacitor_SMD:C_0603_1608Metric_Pad1.05x0.95mm_HandSolder, symbol Device:C
- C56, C57, C60, C61, C64, C65, C68, C69, C72, C76, C81, C82: value 100nF -> 10nF; Digikey 1276-1000-1-ND -> 1276-1009-1-ND
- C59, C62, C63, C66, C67, C70, C71, C74, C75: value 4.7uF -> 10nF; Digikey 1276-1045-1-ND -> 1276-1009-1-ND
- C73, C77, C78, C79, C80, C83: value 100nF -> 47nF; Digikey 1276-1000-1-ND -> 1276-1063-1-ND
Connections:
- net +1V2: now also C63.1, C75.1, C130.1, C136.1, C141.1, C146.1, C148.1, C150.1; no longer C61.1, C62.1, C65.1, C66.1, C70.1, C73.1, C74.1, C77.1, C79.1, C83.1
- net +3V3: now also C61.1, C62.1, C65.1, C66.1, C70.1, C73.1, C74.1, C77.1, C79.1, C83.1, C127.1, C128.1, C129.1, C131.1, C132.1, C133.1, C134.1, C135.1, C137.1, C138.1, C139.1, C140.1, C142.1, C143.1, C144.1, C145.1, C147.1, C149.1, C151.1, C152.1; no longer C63.1, C75.1
- net GND: now also C127.2, C128.2, C129.2, C130.2, C131.2, C132.2, C133.2, C134.2, C135.2, C136.2, C137.2, C138.2, C139.2, C140.2, C141.2, C142.2, C143.2, C144.2, C145.2, C146.2, C147.2, C148.2, C149.2, C150.2, C151.2, C152.2
Other:
- note added: "VCCAUX"
- note added: "VCCINT"
- note added: "VCCO_0"
- note added: "VCCO_1\n"
- note added: "VCCO_2"
- note added: "VCCO_3"
- moved on the sheet: C57, C58, D2, D3, J1, J2, R24, R25, R26, R27, R28, R29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

Commit message: organizacion PCB_V3
Parts:
- removed C127, C129, C130, C131, C132, C133, C135, C136, C137, C141, C142, C146, C147, C148, C149, C83: 47nF, Capacitor_SMD:C_0603_1608Metric_Pad1.05x0.95mm_HandSolder, symbol Device:C
- removed C128, C138, C139, C140, C150, C151: 0.47uF, Capacitor_SMD:C_0603_1608Metric_Pad1.05x0.95mm_HandSolder, symbol Device:C
- removed C134, C143, C144, C145, C152: 4.7uF, Capacitor_SMD:C_0603_1608Metric_Pad1.05x0.95mm_HandSolder, symbol Device:C
- removed C81, C82: 10nF, Capacitor_SMD:C_0603_1608Metric_Pad1.05x0.95mm_HandSolder, symbol Device:C
- C56, C57, C59, C60, C61, C62, C63, C64, C65, C66, C71, C72: value 10nF -> 4.7uF; Digikey 1276-1009-1-ND -> 1276-1045-1-ND
- C67, C68, C69, C70, C74, C75, C76: value 10nF -> 0.47uF; Digikey 1276-1009-1-ND -> 1276-2082-1-ND
- C73, C78, C80: value 47nF -> 0.47uF; Digikey 1276-1063-1-ND -> 1276-2082-1-ND
- C77, C79: value 47nF -> 4.7uF; Digikey 1276-1063-1-ND -> 1276-1045-1-ND
Connections:
- net +1V2: now also C60.1, C66.1, C72.1, C78.1; no longer C58.1, C63.1, C69.1, C75.1
- net +3V3: now also C58.1, C63.1, C69.1, C75.1; no longer C60.1, C66.1, C72.1, C78.1

Commit message: organizacion PCB_V4
Connections:
- net adDA0: now also U4.56 (IO_L30P_GCLK1_D13_2); no longer U4.80 (IO_L46N_1)
- net adDA1: now also U4.57 (IO_L14N_D12_2); no longer U4.79 (IO_L47P_1)
- net adDA2: now also U4.58 (IO_L14P_D11_2); no longer U4.78 (IO_L47N_1)
- net adDA3: now also U4.59 (IO_L13N_D10_2); no longer U4.75 (IO_L74P_1)
- net adDA4: now also U4.60 (IO_L13P_M1_2); no longer U4.74 (IO_L74N_1)
- net adDA5: now also U4.61 (IO_L12N_D2_MISO3_2); no longer U4.70 (IO_L1P_CCLK_2)
- net adDA6: now also U4.62 (IO_L12P_D1_MISO2_2); no longer U4.69 (IO_L1N_M0_CMPMISO_2)
- net adDA7: now also U4.64 (IO_L3N_MOSI_CSI_B_MISO0_2); no longer U4.67 (IO_L2P_CMPCLK_2)
- net adDD0: now also U4.65 (IO_L3P_D0_DIN_MISO_MISO1_2); no longer U4.66 (IO_L2N_CMPMOSI_2)
- net adDD1: now also U4.66 (IO_L2N_CMPMOSI_2); no longer U4.65 (IO_L3P_D0_DIN_MISO_MISO1_2)
- net adDD2: now also U4.67 (IO_L2P_CMPCLK_2); no longer U4.64 (IO_L3N_MOSI_CSI_B_MISO0_2)
- net adDD3: now also U4.69 (IO_L1N_M0_CMPMISO_2); no longer U4.62 (IO_L12P_D1_MISO2_2)
- net adDD4: now also U4.70 (IO_L1P_CCLK_2); no longer U4.61 (IO_L12N_D2_MISO3_2)
- net adDD5: now also U4.74 (IO_L74N_1); no longer U4.60 (IO_L13P_M1_2)
- net adDD6: now also U4.75 (IO_L74P_1); no longer U4.59 (IO_L13N_D10_2)
- net adDD7: now also U4.78 (IO_L47N_1); no longer U4.58 (IO_L14P_D11_2)
- net adDD8: now also U4.79 (IO_L47P_1); no longer U4.57 (IO_L14N_D12_2)
- net adDD9: now also U4.80 (IO_L46N_1); no longer U4.56 (IO_L30P_GCLK1_D13_2)
Changed lines of the file:
@@
 Wire Wire Line
 	12350 3200 12200 3200
-Text GLabel 8900 1900 1    50   Input ~ 0
+Text GLabel 12350 4400 2    50   Input ~ 0
 adDA0
-Text GLabel 9000 1900 1    50   Input ~ 0
+Text GLabel 12350 4300 2    50   Input ~ 0
 adDA1
-Text GLabel 9100 1900 1    50   Input ~ 0
+Text GLabel 12350 4200 2    50   Input ~ 0
 adDA2
 Text Label 6500 7225 1    50   ~ 0
@@
 Wire Wire Line
 	12200 5600 12675 5600
+Text GLabel 12350 3900 2    50   Input ~ 0
+adDA5
+Text GLabel 12350 3800 2    50   Input ~ 0
+adDA6
+Text GLabel 12350 3700 2    50   Input ~ 0
+adDA7
+Text GLabel 12350 3600 2    50   Input ~ 0
+adDD0
+Text GLabel 12350 3500 2    50   Input ~ 0
+adDD1
+Text GLabel 12350 3400 2    50   Input ~ 0
+adDD2
+Text GLabel 12350 3300 2    50   Input ~ 0
+adDD3
 Text GLabel 12350 3200 2    50   Input ~ 0
-adDA5
-Text GLabel 12350 3300 2    50   Input ~ 0
-adDA6
-Text GLabel 12350 3400 2    50   Input ~ 0
-adDA7
-Text GLabel 12350 3500 2    50   Input ~ 0
-adDD0
-Text GLabel 12350 3600 2    50   Input ~ 0
-adDD1
-Text GLabel 12350 3700 2    50   Input ~ 0
-adDD2
-Text GLabel 12350 3800 2    50   Input ~ 0
-adDD3
-Text GLabel 12350 3900 2    50   Input ~ 0
 adDD4
+Text GLabel 9300 1900 1    50   Input ~ 0
+adDD5
+Text GLabel 9200 1900 1    50   Input ~ 0
+adDD6
+Text GLabel 9100 1900 1    50   Input ~ 0
+adDD7
+Text GLabel 9000 1900 1    50   Input ~ 0
+adDD8
+Text GLabel 8900 1900 1    50   Input ~ 0
+adDD9
+Text GLabel 12350 4100 2    50   Input ~ 0
+adDA3
 Text GLabel 12350 4000 2    50   Input ~ 0
-adDD5
-Text GLabel 12350 4100 2    50   Input ~ 0
-adDD6
-Text GLabel 12350 4200 2    50   Input ~ 0
-adDD7
-Text GLabel 12350 4300 2    50   Input ~ 0
-adDD8
-Text GLabel 12350 4400 2    50   Input ~ 0
-adDD9
-Text GLabel 9200 1900 1    50   Input ~ 0
-adDA3
-Text GLabel 9300 1900 1    50   Input ~ 0
 adDA4
 Wire Wire Line

Commit message: PCB route V1
Parts:
- removed C86: 100nF, Capacitor_SMD:C_0603_1608Metric_Pad1.05x0.95mm_HandSolder, symbol Device:C
- added C18: 100nF, Capacitor_SMD:C_0603_1608Metric_Pad1.05x0.95mm_HandSolder, symbol Device:C
Connections:
- net +3V3: now also S1.3, S1.4, S2.3, S2.4; no longer R49.1, R50.1
- net BTN1: now also R49.1; no longer R49.2
- net BTN2: now also R50.1, C18.1; no longer R50.2
- net FPGA_GPIO_01: no longer R35.1
- net FPGA_GPIO_04: now also R35.1
- net GND: now also R49.2, R50.2, C18.2; no longer S1.3, S1.4, S2.3, S2.4
Other:
- moved on the sheet: R49, S1
Changed lines of the file:
@@
-$EndComp
-$Comp
-L power:GND #PWR097
-U 1 1 5D00E8AC
-P 13925 7975
-F 0 "#PWR097" H 13925 7725 50  0001 C CNN
-F 1 "GND" V 13930 7802 50  0000 C CNN
-F 2 "" H 13925 7975 50  0001 C CNN
-F 3 "" H 13925 7975 50  0001 C CNN
-	1    13925 7975
-	1    0    0    -1
 $EndComp
 $Comp
 L Device:R R49
 U 1 1 5D00E8AD
-P 13425 6950
-F 0 "R49" V 13525 6950 50  0000 L CNN
-F 1 "10k" V 13425 6900 50  0000 L CNN
-F 2 "Resistor_SMD:R_0603_1608Metric_Pad1.05x0.95mm_HandSolder" V 13355 6950 50  0001 C CNN
-F 3 "http://www.yageo.com/documents/recent/PYu-RC_Group_51_RoHS_L_10.pdf" H 13425 6950 50  0001 C CNN
-F 4 "311-10KGRCT-ND" V 13425 6950 50  0001 C CNN "Digikey"
-	1    13425 6950
-	0    -1   -1   0
+P 14000 7300
+F 0 "R49" H 14050 7400 50  0000 L CNN
+F 1 "10k" V 14000 7250 50  0000 L CNN
+F 2 "Resistor_SMD:R_0603_1608Metric_Pad1.05x0.95mm_HandSolder" V 13930 7300 50  0001 C CNN
+F 3 "http://www.yageo.com/documents/recent/PYu-RC_Group_51_RoHS_L_10.pdf" H 14000 7300 50  0001 C CNN
+F 4 "311-10KGRCT-ND" V 14000 7300 50  0001 C CNN "Digikey"
+	1    14000 7300
+	1    0    0    -1
 $EndComp
 $Comp
@@
 	1    0    0    -1
 $EndComp
-Wire Wire Line
-	13175 6950 13275 6950
 Text Label 14500 6950 0    50   ~ 0
 BTN1
@@
 	14275 7150 14275 6950
 Wire Wire Line
-	14275 7550 14275 7450
-$Comp
-L power:GND #PWR094
-U 1 1 5D00E8B0
-P 13825 7975
-F 0 "#PWR094" H 13825 7725 50  0001 C CNN
-F 1 "GND" V 13830 7802 50  0000 C CNN
-F 2 "" H 13825 7975 50  0001 C CNN
-F 3 "" H 13825 7975 50  0001 C CNN
-	1    13825 7975
-	1    0    0    -1
-$EndComp
+	14275 7550 14275 7500
 $Comp
 L TL1014BF160QG:TL1014BF160QG S1
 U 1 1 5D00E8B1
-P 13925 7100
-F 0 "S1" V 14279 6778 50  0000 L CNN
-F 1 "TL1014BF160QG" V 14370 6253 50  0000 L CNN
-F 2 "lib:TL1014BF160QG" H 14575 7200 50  0001 L CNN
-F 3 "https://www.e-switch.com/system/asset/product_line/data_sheet/141/TL1014.pdf" H 14575 7100 50  0001 L CNN
-F 4 "EG5042CT-ND" V 13925 7100 50  0001 C CNN "Digikey"
-	1    13925 7100
-	0    1    1    0
-$EndComp
-Text GLabel 13175 6950 0    50   Input ~ 0
+P 13650 7050
+F 0 "S1" H 14000 6800 50  0000 L CNN
+F 1 "TL1014BF160QG" H 13750 7200 50  0000 L CNN
+F 2 "lib:TL1014BF160QG" H 14300 7150 50  0001 L CNN
+F 3 "https://www.e-switch.com/system/asset/product_line/data_sheet/141/TL1014.pdf" H 14300 7050 50  0001 L CNN
+F 4 "EG5042CT-ND" V 13650 7050 50  0001 C CNN "Digikey"
+	1    13650 7050
+	-1   0    0    1
+$EndComp
+Text GLabel 12650 6950 0    50   Input ~ 0
 3V3 FPGA
 Wire Wire Line
 	14500 6950 14275 6950
-Connection ~ 14275 6950
-Wire Wire Line
-	13575 6950 13825 6950
-Wire Wire Line
-	13825 7100 13825 6950
-Connection ~ 13825 6950
-Wire Wire Line
-	13825 6950 13925 6950
-Wire Wire Line
-	13925 7100 13925 6950
-Connection ~ 13925 6950
-Wire Wire Line
-	13925 6950 14275 6950
-Wire Wire Line
-	13825 7975 13825 7900
-Wire Wire Line
-	13925 7900 13925 7975
-Text Notes 12750 6725 0    118  ~ 0
+Text Notes 12550 6600 0    118  ~ 0
 Buttons
-$Comp
-L TL1014BF160QG:TL1014BF160QG S2
-U 1 1 5D03A38F
-P 13925 8525
-F 0 "S2" V 14279 8203 50  0000 L CNN
-F 1 "TL1014BF160QG" V 14370 7678 50  0000 L CNN
-F 2 "lib:TL1014BF160QG" H 14575 8625 50  0001 L CNN
-F 3 "https://www.e-switch.com/system/asset/product_line/data_sheet/141/TL1014.pdf" H 14575 8525 50  0001 L CNN
-F 4 "EG5042CT-ND" V 13925 8525 50  0001 C CNN "Digikey"
-	1    13925 8525
-	0    1    1    0
-$EndComp
-Wire Wire Line
-	13925 8525 13925 8375
-Wire Wire Line
-	13825 9400 13825 9325
-Text GLabel 13175 8375 0    50   Input ~ 0
-3V3 FPGA
-Wire Wire Line
-	14500 8375 14275 8375
-Wire Wire Line
-	13925 8375 14275 8375
-Wire Wire Line
-	14275 8575 14275 8375
-$Comp
-L power:GND #PWR095
-U 1 1 5D03A390
-P 13825 9400
-F 0 "#PWR095" H 13825 9150 50  0001 C CNN
-F 1 "GND" V 13830 9227 50  0000 C CNN
-F 2 "" H 13825 9400 50  0001 C CNN
-F 3 "" H 13825 9400 50  0001 C CNN
-	1    13825 9400
-	1    0    0    -1
-$EndComp
-$Comp
-L power:GND #PWR0100
-U 1 1 5D03A391
-P 14275 8975
-F 0 "#PWR0100" H 14275 8725 50  0001 C CNN
-F 1 "GND" H 14280 8802 50  0000 C CNN
-F 2 "" H 14275 8975 50  0001 C CNN
-F 3 "" H 14275 8975 50  0001 C CNN
-	1    14275 8975
-	1    0    0    -1
-$EndComp
-Connection ~ 13825 8375
-Connection ~ 14275 8375
-Wire Wire Line
-	13175 8375 13275 8375
-Wire Wire Line
-	13825 8525 13825 8375
-$Comp
-L power:GND #PWR098
-U 1 1 5D03A392
-P 13925 9400
-F 0 "#PWR098" H 13925 9150 50  0001 C CNN
-F 1 "GND" V 13930 9227 50  0000 C CNN
-F 2 "" H 13925 9400 50  0001 C CNN
-F 3 "" H 13925 9400 50  0001 C CNN
-	1    13925 9400
-	1    0    0    -1
-$EndComp
-Wire Wire Line
-	13825 8375 13925 8375
 Text Label 14500 8375 0    50   ~ 0
 BTN2
-Wire Wire Line
-	13575 8375 13825 8375
-Wire Wire Line
-	13925 9325 13925 9400
-Connection ~ 13925 8375
-$Comp
-L Device:R R50
-U 1 1 5D03A393
-P 13425 8375
-F 0 "R50" V 13525 8375 50  0000 L CNN
-F 1 "10k" V 13425 8325 50  0000 L CNN
-F 2 "Resistor_SMD:R_0603_1608Metric_Pad1.05x0.95mm_HandSolder" V 13355 8375 50  0001 C CNN
-F 3 "http://www.yageo.com/documents/recent/PYu-RC_Group_51_RoHS_L_10.pdf" H 13425 8375 50  0001 C CNN
-F 4 "311-10KGRCT-ND" V 13425 8375 50  0001 C CNN "Digikey"
-	1    13425 8375
-	0    -1   -1   0
-$EndComp
-$Comp
-L Device:C C86
-U 1 1 5D03A394
-P 14275 8725
-F 0 "C86" H 14375 8825 50  0000 C CNN
-F 1 "100nF" H 14425 8625 50  0000 C CNN
-F 2 "Capacitor_SMD:C_0603_1608Metric_Pad1.05x0.95mm_HandSolder" H 14313 8575 50  0001 C CNN
-F 3 "http://www.samsungsem.com/kr/support/product-search/mlcc/__icsFiles/afieldfile/2018/07/24/CL10B104KB8NNNC.pdf" H 14275 8725 50  0001 C CNN
-F 4 "1276-1000-1-ND" H 14275 8725 50  0001 C CNN "Digikey"
-	1    14275 8725
-	1    0    0    -1
-$EndComp
-Wire Wire Line
-	14275 8975 14275 8875
 Text Label 7550 10025 0    50   ~ 0
 FMC_CLK
@@
 FPGA_GPIO_06
 Text Label 7075 9450 2    50   ~ 0
-FPGA_GPIO_01
-Text Label 7025 10975 2    50   ~ 0
+FPGA_GPIO_04
+Text Label 6825 10975 2    50   ~ 0
 SCL_I2C
 Text Label 5025 3950 0    50   ~ 0
@@
 Wire Wire Line
 	7025 10875 6400 10875
-Wire Wire Line
-	5950 10975 7025 10975
 Wire Wire Line
 	5075 10575 4500 10575
@@
 Text GLabel 8000 10625 2    50   Output ~ 0
 FMC_NBL1
-Text Label 4375 10975 0    50   ~ 0
+Text Label 4775 10975 0    50   ~ 0
 SDA_I2C
-Wire Wire Line
-	5450 10975 4375 10975
 Text Notes 1100 1600 0    50   ~ 0
 VCCINT
@@
 	1    0    0    -1
 $EndComp
+Wire Wire Line
+	12850 7050 12750 7050
+Wire Wire Line
+	14000 7450 14000 7500
+Wire Wire Line
+	14000 7500 14275 7500
+Connection ~ 14275 7500
+Wire Wire Line
+	14275 7500 14275 7450
+Wire Wire Line
+	13650 6950 13750 6950
+Connection ~ 14275 6950
+Wire Wire Line
+	13650 7050 13750 7050
+Wire Wire Line
+	13750 7050 13750 6950
+Connection ~ 13750 6950
+Wire Wire Line
+	13750 6950 14000 6950
+Wire Wire Line
+	14000 7150 14000 6950
+Connection ~ 14000 6950
+Wire Wire Line
+	14000 6950 14275 6950
+Wire Wire Line
+	12750 7050 12750 6950
+Wire Wire Line
+	12750 6950 12650 6950
+Wire Wire Line
+	12850 6950 12750 6950
+Connection ~ 12750 6950
+$Comp
+L Device:R R50
+U 1 1 5D057BA2
+P 14000 8725
+F 0 "R50" H 14050 8825 50  0000 L CNN
+F 1 "10k" V 14000 8675 50  0000 L CNN
+F 2 "Resistor_SMD:R_0603_1608Metric_Pad1.05x0.95mm_HandSolder" V 13930 8725 50  0001 C CNN
+F 3 "http://www.yageo.com/documents/recent/PYu-RC_Group_51_RoHS_L_10.pdf" H 14000 8725 50  0001 C CNN
+F 4 "311-10KGRCT-ND" V 14000 8725 50  0001 C CNN "Digikey"
+	1    14000 8725
+	1    0    0    -1
+$EndComp
+$Comp
+L power:GND #PWR06
+U 1 1 5D057BAA
+P 14275 8975
+F 0 "#PWR06" H 14275 8725 50  0001 C CNN
+F 1 "GND" H 14280 8802 50  0000 C CNN
+F 2 "" H 14275 8975 50  0001 C CNN
+F 3 "" H 14275 8975 50  0001 C CNN
+	1    14275 8975
+	1    0    0    -1
+$EndComp
+$Comp
+L Device:C C18
+U 1 1 5D057BB5
+P 14275 8725
+F 0 "C18" H 14375 8825 50  0000 C CNN
+F 1 "100nF" H 14425 8625 50  0000 C CNN
+F 2 "Capacitor_SMD:C_0603_1608Metric_Pad1.05x0.95mm_HandSolder" H 14313 8575 50  0001 C CNN
+F 3 "http://www.samsungsem.com/kr/support/product-search/mlcc/__icsFiles/afieldfile/2018/07/24/CL10B104KB8NNNC.pdf" H 14275 8725 50  0001 C CNN
+F 4 "1276-1000-1-ND" H 14275 8725 50  0001 C CNN "Digikey"
+	1    14275 8725
+	1    0    0    -1
+$EndComp
+Wire Wire Line
+	14275 8575 14275 8375
+Wire Wire Line
+	14275 8975 14275 8925
+$Comp
+L TL1014BF160QG:TL1014BF160QG S2
+U 1 1 5D057BC6
+P 13650 8475
+F 0 "S2" H 14000 8225 50  0000 L CNN
+F 1 "TL1014BF160QG" H 13750 8625 50  0000 L CNN
+F 2 "lib:TL1014BF160QG" H 14300 8575 50  0001 L CNN
+F 3 "https://www.e-switch.com/system/asset/product_line/data_sheet/141/TL1014.pdf" H 14300 8475 50  0001 L CNN
+F 4 "EG5042CT-ND" V 13650 8475 50  0001 C CNN "Digikey"
+	1    13650 8475
+	-1   0    0    1
+$EndComp
+Text GLabel 12650 8375 0    50   Input ~ 0
+3V3 FPGA
+Wire Wire Line
+	14500 8375 14275 8375
+Wire Wire Line
+	12850 8475 12750 8475
+Wire Wire Line
+	14000 8875 14000 8925
+Wire Wire Line
+	14000 8925 14275 8925
+Connection ~ 14275 8925
+Wire Wire Line
+	14275 8925 14275 8875
+Wire Wire Line
+	13650 8375 13750 8375
+Connection ~ 14275 8375
+Wire Wire Line
+	13650 8475 13750 8475
+Wire Wire Line
+	13750 8475 13750 8375
+Connection ~ 13750 8375
+Wire Wire Line
+	13750 8375 14000 8375
+Wire Wire Line
+	14000 8575 14000 8375
+Connection ~ 14000 8375
+Wire Wire Line
+	14000 8375 14275 8375
+Wire Wire Line
+	12750 8475 12750 8375
+Wire Wire Line
+	12750 8375 12650 8375
+Wire Wire Line
+	12850 8375 12750 8375
+Connection ~ 12750 8375
+Text GLabel 6875 10975 2    50   Input ~ 0
+I2C_SCL
+Text GLabel 4700 10975 0    50   Input ~ 0
+I2C_SDA
+Wire Wire Line
+	5950 10975 6875 10975
+Wire Wire Line
+	4700 10975 5450 10975
 $EndSCHEMATC

Commit message: PCB route V3
Changed lines of the file:
@@
 	9300 8525 9800 8525
 Wire Notes Line
-	7200 7525 7200 11275
-Wire Notes Line
-	11350 7525 7200 7525
-Text Notes 7900 7725 0    50   ~ 0
+	11825 7850 7675 7850
+Text Notes 8375 8050 0    50   ~ 0
 BUS DATA-ADDRESS-CONTROL \nPROC<->FPGA\n
 Text Label 8200 7150 1    50   ~ 0
@@
 Text Label 5100 4550 0    50   ~ 0
 FMC_CLK
-Text Label 5100 4350 0    50   ~ 0
-FMC_NWE
-Text Label 5100 4150 0    50   ~ 0
-FMC_NE1
 Text Label 5100 4450 0    50   ~ 0
 FMC_NOE
@@
 	8200 7150 8200 6650
 Wire Notes Line
-	11350 11275 11350 7525
+	10425 11600 10425 7850
 Wire Notes Line
 	7200 11275 11350 11275
@@
 Wire Wire Line
 	5100 4250 5600 4250
-Text Label 5100 4250 0    50   ~ 0
-FMC_NWAIT
 Wire Wire Line
 	8800 7150 8800 6650
@@
 Text Label 7550 10025 0    50   ~ 0
 FMC_CLK
-Text Label 7550 10225 0    50   ~ 0
-FMC_NWE
-Text Label 7550 10325 0    50   ~ 0
-FMC_NWAIT
-Text Label 7550 10425 0    50   ~ 0
-FMC_NE1
 Text Label 7550 10125 0    50   ~ 0
 FMC_NOE
@@
 Wire Wire Line
 	8000 10125 7550 10125
-Text GLabel 8000 9925 2    50   Output ~ 0
+Text GLabel 8000 9925 2    50   Input ~ 0
 FMC_NL
-Text GLabel 8000 10025 2    50   Output ~ 0
+Text GLabel 8000 10025 2    50   Input ~ 0
 FMC_CLK
-Text GLabel 8000 10125 2    50   Output ~ 0
+Text GLabel 8000 10125 2    50   Input ~ 0
 FMC_NOE
-Text GLabel 8000 10225 2    50   Output ~ 0
+Text GLabel 8000 10225 2    50   Input ~ 0
 FMC_NWE
-Text GLabel 8000 10325 2    50   Output ~ 0
+Text GLabel 8000 10325 2    50   Input ~ 0
 FMC_NWAIT
-Text GLabel 8000 10425 2    50   Output ~ 0
-FMC_NE1
-Text GLabel 8000 10525 2    50   Output ~ 0
+Text GLabel 8000 10525 2    50   Input ~ 0
 FMC_NBL0
-Text GLabel 8000 10625 2    50   Output ~ 0
+Text GLabel 8000 10625 2    50   Input ~ 0
 FMC_NBL1
 Text Label 4775 10975 0    50   ~ 0
@@
 Wire Wire Line
 	4700 10975 5450 10975
+Text Label 7550 10225 0    50   ~ 0
+FMC_NWE
+Text Label 5100 4350 0    50   ~ 0
+FMC_NWE
+Text GLabel 8000 10425 2    50   Input ~ 0
+FMC_NE1
+Text Label 5100 4250 0    50   ~ 0
+FMC_NWAIT
+Text Label 5100 4150 0    50   ~ 0
+FMC_NE1
+Text Label 7550 10425 0    50   ~ 0
+FMC_NE1
+Text Label 7550 10325 0    50   ~ 0
+FMC_NWAIT
+Text GLabel 5100 4450 0    50   Input ~ 0
+FMC_NOE
+Text GLabel 5100 4550 0    50   Input ~ 0
+FMC_CLK
+Text GLabel 5100 4350 0    50   Input ~ 0
+FMC_NWE
+Text GLabel 5100 4250 0    50   Input ~ 0
+FMC_NWAIT
+Text GLabel 5100 4150 0    50   Input ~ 0
+FMC_NE1
+Text GLabel 5100 2850 0    50   Input ~ 0
+FMC_NBL0
+Text GLabel 5100 2750 0    50   Input ~ 0
+FMC_NBL1
+Text GLabel 5100 3150 0    50   Input ~ 0
+FMC_NL
+Text GLabel 5100 4750 0    50   Input ~ 0
+FMC_D2
+Text GLabel 5100 4650 0    50   Input ~ 0
+FMC_D3
+Text GLabel 12700 4900 2    50   Input ~ 0
+FMC_D7
+Text GLabel 12700 4600 2    50   Input ~ 0
+FMC_D4
+Text GLabel 12700 4800 2    50   Input ~ 0
+FMC_D6
+Text GLabel 12700 4700 2    50   Input ~ 0
+FMC_D5
+Text GLabel 12700 5300 2    50   Input ~ 0
+FMC_D11
+Text GLabel 12700 5000 2    50   Input ~ 0
+FMC_D8
+Text GLabel 12700 5200 2    50   Input ~ 0
+FMC_D10
+Text GLabel 12700 5100 2    50   Input ~ 0
+FMC_D9
+Text GLabel 8700 7150 3    50   Input ~ 0
+FMC_D15
+Text GLabel 12700 5400 2    50   Input ~ 0
+FMC_D12
+Text GLabel 8800 7150 3    50   Input ~ 0
+FMC_D14
+Text GLabel 8900 7150 3    50   Input ~ 0
+FMC_D13
+Text GLabel 8300 7150 3    50   Input ~ 0
+FMC_D1
+Text GLabel 8200 7150 3    50   Input ~ 0
+FMC_D0
+Text GLabel 8600 7150 3    50   Input ~ 0
+FMC_A16
+Text GLabel 8500 7150 3    50   Input ~ 0
+FMC_A17
+Text GLabel 8400 7150 3    50   Input ~ 0
+FMC_A18
+Text GLabel 7300 1600 1    50   Input ~ 0
+FMC_A19
+Text GLabel 7400 1600 1    50   Input ~ 0
+FMC_A20
+Text GLabel 7500 1600 1    50   Input ~ 0
+FMC_A21
+Text GLabel 7600 1600 1    50   Input ~ 0
+FMC_A22
+Text GLabel 7200 1600 1    50   Input ~ 0
+FMC_A23
+Text GLabel 8000 7150 3    50   Input ~ 0
+FMC_A15
+Text GLabel 8100 7150 3    50   Input ~ 0
+FMC_A14
 $EndSCHEMATC
