File: HW/shield_SDR_UN/FPGA.sch (KiCad schematic (older format))
At the start: 68 parts, among them J1 Conn_02x09_Odd_Even, J2 Conn_02x08_Odd_Even, U4 XC6SLX9-2TQG144C, X2 ASE-xxxMHz

Commit message: PCB routing
Parts:
- added R64, R65: 1.5k, Resistor_SMD:R_0603_1608Metric_Pad1.05x0.95mm_HandSolder, symbol Device:R
Connections:
- net +3V3: now also U4.60 (IO_L13P_M1_2), U4.69 (IO_L1N_M0_CMPMISO_2)
- net adDA4: now also U4.61 (IO_L12N_D2_MISO3_2); no longer U4.60 (IO_L13P_M1_2)
- net adDA5: now also U4.62 (IO_L12P_D1_MISO2_2); no longer U4.61 (IO_L12N_D2_MISO3_2)
- net adDA6: now also U4.64 (IO_L3N_MOSI_CSI_B_MISO0_2); no longer U4.62 (IO_L12P_D1_MISO2_2)
- net adDA7: now also U4.65 (IO_L3P_D0_DIN_MISO_MISO1_2); no longer U4.64 (IO_L3N_MOSI_CSI_B_MISO0_2)
- net adDD0: now also U4.66 (IO_L2N_CMPMOSI_2); no longer U4.65 (IO_L3P_D0_DIN_MISO_MISO1_2)
- net adDD1: now also U4.67 (IO_L2P_CMPCLK_2); no longer U4.66 (IO_L2N_CMPMOSI_2)
- net adDD2: now also U4.70 (IO_L1P_CCLK_2); no longer U4.67 (IO_L2P_CMPCLK_2)
- net adDD3: now also U4.74 (IO_L74N_1); no longer U4.69 (IO_L1N_M0_CMPMISO_2)
- net adDD4: now also U4.75 (IO_L74P_1); no longer U4.70 (IO_L1P_CCLK_2)
- net adDD5: now also U4.78 (IO_L47N_1); no longer U4.74 (IO_L74N_1)
- net adDD6: now also U4.79 (IO_L47P_1); no longer U4.75 (IO_L74P_1)
- net adDD7: now also U4.80 (IO_L46N_1); no longer U4.78 (IO_L47N_1)
- net adDD8: now also U4.81 (IO_L46P_1); no longer U4.79 (IO_L47P_1)
- net adDD9: now also U4.82 (IO_L45N_1); no longer U4.80 (IO_L46N_1)
- no-connect marks 19 -> 17
Changed lines of the file:
@@
 	12200 4100 12350 4100
 Wire Wire Line
-	12350 4000 12200 4000
-Wire Wire Line
 	12200 3900 12350 3900
 Wire Wire Line
@@
 Wire Wire Line
 	12350 3400 12200 3400
-Wire Wire Line
-	12200 3300 12350 3300
 Wire Wire Line
 	12350 3200 12200 3200
@@
 Wire Wire Line
 	12200 5600 12675 5600
-Text GLabel 12350 3900 2    50   Input ~ 0
+Text GLabel 12350 3800 2    50   Input ~ 0
 adDA5
-Text GLabel 12350 3800 2    50   Input ~ 0
+Text GLabel 12350 3700 2    50   Input ~ 0
 adDA6
-Text GLabel 12350 3700 2    50   Input ~ 0
+Text GLabel 12350 3600 2    50   Input ~ 0
 adDA7
-Text GLabel 12350 3600 2    50   Input ~ 0
+Text GLabel 12350 3500 2    50   Input ~ 0
 adDD0
-Text GLabel 12350 3500 2    50   Input ~ 0
+Text GLabel 12350 3400 2    50   Input ~ 0
 adDD1
-Text GLabel 12350 3400 2    50   Input ~ 0
+Text GLabel 12350 3200 2    50   Input ~ 0
 adDD2
-Text GLabel 12350 3300 2    50   Input ~ 0
+Text GLabel 9300 1900 1    50   Input ~ 0
 adDD3
-Text GLabel 12350 3200 2    50   Input ~ 0
+Text GLabel 9200 1900 1    50   Input ~ 0
 adDD4
-Text GLabel 9300 1900 1    50   Input ~ 0
+Text GLabel 9100 1900 1    50   Input ~ 0
 adDD5
-Text GLabel 9200 1900 1    50   Input ~ 0
+Text GLabel 9000 1900 1    50   Input ~ 0
 adDD6
-Text GLabel 9100 1900 1    50   Input ~ 0
+Text GLabel 8900 1900 1    50   Input ~ 0
 adDD7
-Text GLabel 9000 1900 1    50   Input ~ 0
+Text GLabel 8800 1900 1    50   Input ~ 0
 adDD8
-Text GLabel 8900 1900 1    50   Input ~ 0
+Text GLabel 8700 1900 1    50   Input ~ 0
 adDD9
 Text GLabel 12350 4100 2    50   Input ~ 0
 adDA3
-Text GLabel 12350 4000 2    50   Input ~ 0
+Text GLabel 12350 3900 2    50   Input ~ 0
 adDA4
 Wire Wire Line
-	9300 1900 9300 2100
-Wire Wire Line
-	9200 2100 9200 1900
+	9100 1900 9100 2100
+Wire Wire Line
+	9000 2100 9000 1900
+Wire Wire Line
+	8700 1900 8700 2100
+Wire Wire Line
+	8800 1900 8800 2100
 Wire Wire Line
 	8900 1900 8900 2100
-Wire Wire Line
-	9000 1900 9000 2100
-Wire Wire Line
-	9100 1900 9100 2100
 Text GLabel 8400 1875 1    50   Input ~ 0
 GCK1
@@
 NoConn ~ 8300 2100
 NoConn ~ 8600 2100
-NoConn ~ 8700 2100
-NoConn ~ 8800 2100
 NoConn ~ 5600 5250
 NoConn ~ 5600 5150
@@
 Text GLabel 8100 7150 3    50   Input ~ 0
 FMC_A14
+Wire Wire Line
+	12200 3300 12675 3300
+Wire Wire Line
+	12200 4000 12675 4000
+Text Label 12675 3300 0    50   ~ 0
+FPGA_M0
+Text Label 12675 4000 0    50   ~ 0
+FPGA_M1
+$Comp
+L Device:R R64
+U 1 0 5CFFF774
+P 13975 5775
+F 0 "R64" H 14025 5825 50  0000 L CNN
+F 1 "1.5k" V 13975 5675 50  0000 L CNN
+F 2 "Resistor_SMD:R_0603_1608Metric_Pad1.05x0.95mm_HandSolder" V 13905 5775 50  0001 C CNN
+F 3 "http://www.yageo.com/documents/recent/PYu-RC_Group_51_RoHS_L_10.pdf" H 13975 5775 50  0001 C CNN
+F 4 "311-1.5KGRCT-ND" V 13975 5775 50  0001 C CNN "Digikey"
+	1    13975 5775
+	1    0    0    -1
+$EndComp
+$Comp
+L power:GND #PWR071
+U 1 1 5D00A8FA
+P 13975 6000
+F 0 "#PWR071" H 13975 5750 50  0001 C CNN
+F 1 "GND" H 13975 5850 50  0000 C CNN
+F 2 "" H 13975 6000 50  0001 C CNN
+F 3 "" H 13975 6000 50  0001 C CNN
+	1    13975 6000
+	1    0    0    -1
+$EndComp
+$Comp
+L power:GND #PWR072
+U 1 1 5D00AB0A
+P 14200 6000
+F 0 "#PWR072" H 14200 5750 50  0001 C CNN
+F 1 "GND" H 14200 5850 50  0000 C CNN
+F 2 "" H 14200 6000 50  0001 C CNN
+F 3 "" H 14200 6000 50  0001 C CNN
+	1    14200 6000
+	1    0    0    -1
+$EndComp
+Text GLabel 14350 5500 2    50   Input ~ 0
+3V3 FPGA
+Wire Wire Line
+	13975 5925 13975 6000
+Wire Wire Line
+	14200 5925 14200 6000
+Wire Wire Line
+	14200 5625 14200 5500
+Wire Wire Line
+	14200 5500 14350 5500
+Wire Wire Line
+	14200 5500 13975 5500
+Wire Wire Line
+	13975 5500 13975 5625
+Connection ~ 14200 5500
+Text Label 14200 5500 1    50   ~ 0
+FPGA_M0
+Text Label 13975 5500 1    50   ~ 0
+FPGA_M1
+$Comp
+L Device:R R65
+U 1 0 5D052DB9
+P 14200 5775
+F 0 "R65" H 14250 5825 50  0000 L CNN
+F 1 "1.5k" V 14200 5675 50  0000 L CNN
+F 2 "Resistor_SMD:R_0603_1608Metric_Pad1.05x0.95mm_HandSolder" V 14130 5775 50  0001 C CNN
+F 3 "http://www.yageo.com/documents/recent/PYu-RC_Group_51_RoHS_L_10.pdf" H 14200 5775 50  0001 C CNN
+F 4 "311-1.5KGRCT-ND" V 14200 5775 50  0001 C CNN "Digikey"
+	1    14200 5775
+	1    0    0    -1
+$EndComp
+Wire Wire Line
+	9300 2100 9300 1900
+Wire Wire Line
+	9200 1900 9200 2100
 $EndSCHEMATC

Commit message: PCB_VERSION2
Connections:
- net +3V3: now also R64.1, R65.1
- net GND: now also R64.2, R65.2
Changed lines of the file:
@@
 $Comp
 L Device:R R64
-U 1 0 5CFFF774
+U 1 1 5CFFF774
 P 13975 5775
 F 0 "R64" H 14025 5825 50  0000 L CNN
@@
 $Comp
 L Device:R R65
-U 1 0 5D052DB9
+U 1 1 5D052DB9
 P 14200 5775
 F 0 "R65" H 14250 5825 50  0000 L CNN
