File: HW/shield_SDR_UN/shield_SDR_UN.kicad_pcb (KiCad board)
At the start: 2 copper layers, 243 parts, among them J1 Conn_02x09_Odd_Even, J2 Conn_02x08_Odd_Even, J3 Conn_02x10_Top_Bottom, J4 USB_B_Micro, J5 USB_A, J6 Conn_02x06_Odd_Even, P1 GSG-RF-CONN, P2 GSG-RF-CONN, Q1 MOSFET_P, T1 BALUN, T2 BALUN, U1 MAX2830, U2 SI5351C, U3 MAX5864, U4 XC6SLX9-2TQG144C, U5 STM32F722ZET, U6 ZLDO1117G33TA, U7 ZLDO1117G33TA, U8 ZLDO1117G12TA, U9 OMEGA_2, X1 GSG-XTAL4PIN, X2 ASE-xxxMHz, X3 CRYSTAL, X4 GSG-XTAL4PIN

Commit message: Omega 2 PCB
Parts:
- D10: footprint Diode_SMD:D_SMA_Handsoldering -> Diode_SMD:D_SOD-123
- moved C18 302.3 mm to (395.3, -80.5)
- moved CA1 294.2 mm to (404.0, -80.5)
- moved C27 293.9 mm to (394.2, -68.0)
- moved U9 293.3 mm to (264.4, 122.1), turned to 180 degrees
- moved R4 290.0 mm to (404.0, -78.0)
- moved C35 288.1 mm to (386.6, -78.0)
- moved C24 287.6 mm to (389.8, -73.0)
- moved U3 287.4 mm to (374.8, -76.8)
- moved R14 284.7 mm to (398.5, -66.3)
- moved R15 284.2 mm to (393.8, -60.4)
- moved C29 281.8 mm to (386.2, -75.5)
- moved C16 281.4 mm to (380.8, -65.6)
- moved S5 281.0 mm to (235.8, 148.7)
- moved C3 280.4 mm to (381.9, -77.6)
- moved C4 280.3 mm to (386.6, -80.5)
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Connections:
- net /FPGA/FPGA_JTDO renamed /FPGA_JTDO
- net /omega_2/BOOT_0 renamed /BOOT_0
- net /omega_2/OMG_JNRST renamed /OMG_JNRST
- net /omega_2/OMG_JTCK renamed /OMG_JTCK
- net /omega_2/OMG_JTDI renamed /OMG_JTDI
- net /omega_2/OMG_JTMS renamed /OMG_JTMS
- net /omega_2/OMG_JTRST renamed /OMG_JTRST
- net /proc/STM_JTDO renamed /STM_JTDO
- J2 pad 13: /omega_2/SDA_I2C -> I2C_SDA
- J2 pad 14: /omega_2/SCL_I2C -> I2C_SCL
- R3 pad 1: /proc/SPI1_MISO -> SPI1_MISO
- R4 pad 2: /omega_2/I2C1_SDA -> I2C_SCL
- R5 pad 2: /omega_2/I2C1_SCL -> I2C_SDA
- U1 pad 19: /proc/SPI1_MISO -> SPI1_MISO
- U2 pad 4: /omega_2/I2C1_SCL -> I2C_SDA
- U2 pad 5: /omega_2/I2C1_SDA -> I2C_SCL
- U3 pad 34: /proc/SPI1_MISO -> SPI1_MISO
- U4 pad 100: /proc/FMC_A20 -> FMC_A20
- U4 pad 102: /proc/FMC_A23 -> FMC_A23
- U4 pad 116: /proc/FMC_NL -> FMC_NL
- U4 pad 137: /proc/FMC_CLK -> FMC_CLK
- U4 pad 138: /proc/FMC_D3 -> FMC_D3
- U4 pad 22: /proc/FMC_A15 -> FMC_A15
- U4 pad 23: /proc/FMC_A14 -> FMC_A14
- U4 pad 26: /proc/FMC_D0 -> FMC_D0
- U4 pad 33: /proc/FMC_D14 -> FMC_D14
- U4 pad 34: /proc/FMC_D13 -> FMC_D13
- U4 pad 48: /proc/FMC_D6 -> FMC_D6
- U5 pad 114: /FPGA/FMC_D2 -> FMC_D2
- U5 pad 118: /FPGA/FMC_NOE -> FMC_NOE
- U5 pad 119: /FPGA/FMC_NWE -> FMC_NWE
- U5 pad 122: /FPGA/FMC_NWAIT -> FMC_NWAIT
- U5 pad 123: /FPGA/FMC_NE1 -> FMC_NE1
- U5 pad 141: /FPGA/FMC_NBL0 -> FMC_NBL0
- U5 pad 142: /FPGA/FMC_NBL1 -> FMC_NBL1
- U5 pad 2: /FPGA/FMC_A19 -> FMC_A19
- U5 pad 4: /FPGA/FMC_A21 -> FMC_A21
- U5 pad 40: /rf_front_end/SPI1_CS_RF -> SPI1_CS_RF
- U5 pad 41: /rf_front_end/SPI1_SCK -> SPI1_SCK
- U5 pad 43: /rf_front_end/SPI1_MOSI -> SPI1_MOSI
- U5 pad 44: /rf_front_end/SPI1_CS_AD -> SPI1_CS_AD
- U5 pad 5: /FPGA/FMC_A22 -> FMC_A22
- U5 pad 58: /FPGA/FMC_D4 -> FMC_D4
- U5 pad 59: /FPGA/FMC_D5 -> FMC_D5
- U5 pad 63: /FPGA/FMC_D7 -> FMC_D7
- U5 pad 64: /FPGA/FMC_D8 -> FMC_D8
- U5 pad 65: /FPGA/FMC_D9 -> FMC_D9
- U5 pad 66: /FPGA/FMC_D10 -> FMC_D10
- U5 pad 67: /FPGA/FMC_D11 -> FMC_D11
- U5 pad 68: /FPGA/FMC_D12 -> FMC_D12
- U5 pad 79: /FPGA/FMC_D15 -> FMC_D15
- U5 pad 80: /FPGA/FMC_A16 -> FMC_A16
- U5 pad 81: /FPGA/FMC_A17 -> FMC_A17
- U5 pad 82: /FPGA/FMC_A18 -> FMC_A18
- U5 pad 86: /FPGA/FMC_D1 -> FMC_D1
Other:
- board outline added: 100 x 100 mm

Commit message: organizacion PCB_V2
Parts:
- C56, C57, C58, C59, C60, C61, C62, C63, C64, C65, C66, C67, C68, C69, C70, C71, C72, C73, C74, C75, C76, C78, C80, C82, U4: moved to B.Cu
- C77, C79, C81, C83: value 100nF -> 4.7uF; moved to B.Cu
- moved C79 312.6 mm to (54.0, 146.5), turned to 180 degrees
- moved C81 310.9 mm to (76.8, 157.0), turned to 270 degrees
- moved C64 305.4 mm to (70.7, 157.0), turned to 270 degrees
- moved C71 304.0 mm to (54.0, 137.6), turned to 180 degrees
- moved C78 301.8 mm to (54.0, 148.0), turned to 180 degrees
- moved C80 301.7 mm to (78.3, 157.0), turned to 270 degrees
- moved J1 299.9 mm to (18.0, 131.6)
- moved C68 299.8 mm to (54.0, 139.1), turned to 180 degrees
- moved C75 296.6 mm to (76.0, 124.5), turned to 90 degrees
- moved C74 294.2 mm to (73.0, 124.5), turned to 90 degrees
- moved C63 294.0 mm to (89.3, 152.2)
- moved C66 292.1 mm to (73.8, 157.0), turned to 270 degrees
- moved C57 290.3 mm to (89.4, 141.0)
- moved C65 289.9 mm to (72.2, 157.0), turned to 270 degrees
- moved C76 288.7 mm to (68.3, 124.5), turned to 90 degrees
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Connections:
- net /BOOT_0 renamed /omega_2/BOOT_0
- net /FPGA_JTDO renamed /FPGA/FPGA_JTDO
- net /OMG_JNRST renamed /omega_2/OMG_JNRST
- net /OMG_JTCK renamed /omega_2/OMG_JTCK
- net /OMG_JTDI renamed /omega_2/OMG_JTDI
- net /OMG_JTMS renamed /omega_2/OMG_JTMS
- net /OMG_JTRST renamed /omega_2/OMG_JTRST
- net /STM_JTDO renamed /proc/STM_JTDO
- C77 pad 1: 1V2 FPGA -> 3V3 FPGA
- C79 pad 1: 1V2 FPGA -> 3V3 FPGA
- C81 pad 1: 1V2 FPGA -> 3V3 FPGA
- C83 pad 1: 1V2 FPGA -> 3V3 FPGA
- J2 pad 13: I2C_SDA -> /omega_2/SDA_I2C
- J2 pad 14: I2C_SCL -> /omega_2/SCL_I2C
- J6 pad 10: /omega_2/O_SPI_MISO -> /omega_2/SER_TX0
- J6 pad 3: I2C_SCL -> /omega_2/O_SPI_CS1
- J6 pad 4: /omega_2/O_SPI_CS1 -> /omega_2/O_SPI_CLK
- J6 pad 5: I2C_SDA -> /omega_2/O_SPI_MOSI
- J6 pad 6: /omega_2/O_SPI_CLK -> /omega_2/O_SPI_MISO
- J6 pad 7: /omega_2/SER_RX0 -> I2C_SDA
- J6 pad 8: /omega_2/O_SPI_MOSI -> I2C_SCL
- J6 pad 9: /omega_2/SER_TX0 -> /omega_2/SER_RX0
- R3 pad 2: SPI1_MOSI -> /proc/SPI1_MOSI
- R4 pad 2: I2C_SCL -> /omega_2/I2C1_SDA
- R5 pad 2: I2C_SDA -> /omega_2/I2C1_SCL
- U1 pad 18: SPI1_SCK -> /proc/SPI1_SCK
- U2 pad 4: I2C_SDA -> /omega_2/I2C1_SCL
- U2 pad 5: I2C_SCL -> /omega_2/I2C1_SDA
- U3 pad 35: SPI1_SCK -> /proc/SPI1_SCK
- U4 pad 100: FMC_A20 -> /proc/FMC_A20
- U4 pad 101: FMC_A19 -> /proc/FMC_A19
- U4 pad 102: FMC_A23 -> /proc/FMC_A23
- U4 pad 112: FMC_NBL0 -> /proc/FMC_NBL0
- U4 pad 116: FMC_NL -> /proc/FMC_NL
- U4 pad 132: FMC_NWAIT -> /proc/FMC_NWAIT
- U4 pad 133: FMC_NWE -> /proc/FMC_NWE
- U4 pad 137: FMC_CLK -> /proc/FMC_CLK
- U4 pad 27: FMC_A18 -> /proc/FMC_A18
- U4 pad 29: FMC_A17 -> /proc/FMC_A17
- U4 pad 32: FMC_D15 -> /proc/FMC_D15
- U4 pad 41: FMC_D12 -> /proc/FMC_D12
- U4 pad 45: FMC_D9 -> /proc/FMC_D9
- U4 pad 46: FMC_D8 -> /proc/FMC_D8
- U4 pad 47: FMC_D7 -> /proc/FMC_D7
- U5 pad 114: FMC_D2 -> /FPGA/FMC_D2
- U5 pad 115: FMC_D3 -> /FPGA/FMC_D3
- U5 pad 118: FMC_NOE -> /FPGA/FMC_NOE
- U5 pad 123: FMC_NE1 -> /FPGA/FMC_NE1
- U5 pad 142: FMC_NBL1 -> /FPGA/FMC_NBL1
- U5 pad 4: FMC_A21 -> /FPGA/FMC_A21
- U5 pad 40: SPI1_CS_RF -> /rf_front_end/SPI1_CS_RF
- U5 pad 42: SPI1_MISO -> /rf_front_end/SPI1_MISO
- U5 pad 44: SPI1_CS_AD -> /rf_front_end/SPI1_CS_AD
- U5 pad 5: FMC_A22 -> /FPGA/FMC_A22
- U5 pad 58: FMC_D4 -> /FPGA/FMC_D4
- U5 pad 59: FMC_D5 -> /FPGA/FMC_D5
- U5 pad 60: FMC_D6 -> /FPGA/FMC_D6
- U5 pad 66: FMC_D10 -> /FPGA/FMC_D10
- U5 pad 67: FMC_D11 -> /FPGA/FMC_D11
- U5 pad 77: FMC_D13 -> /FPGA/FMC_D13
- U5 pad 78: FMC_D14 -> /FPGA/FMC_D14
- U5 pad 80: FMC_A16 -> /FPGA/FMC_A16
- U5 pad 85: FMC_D0 -> /FPGA/FMC_D0
- U5 pad 86: FMC_D1 -> /FPGA/FMC_D1
- U5 pad 89: FMC_A14 -> /FPGA/FMC_A14
- U5 pad 90: FMC_A15 -> /FPGA/FMC_A15

Commit message: ADC PCB
Parts:
- added C127: 47nF, Capacitor_SMD:C_0603_1608Metric_Pad1.05x0.95mm_HandSolder, F.Cu at (183.2, -24.2)
- added C128: 0.47uF, Capacitor_SMD:C_0603_1608Metric_Pad1.05x0.95mm_HandSolder, F.Cu at (187.6, -26.7)
- added C129: 47nF, Capacitor_SMD:C_0603_1608Metric_Pad1.05x0.95mm_HandSolder, B.Cu at (283.5, 86.4)
- added C130: 47nF, Capacitor_SMD:C_0603_1608Metric_Pad1.05x0.95mm_HandSolder, F.Cu at (183.2, -21.7)
- added C131: 47nF, Capacitor_SMD:C_0603_1608Metric_Pad1.05x0.95mm_HandSolder, F.Cu at (178.9, -16.7)
- added C132: 47nF, Capacitor_SMD:C_0603_1608Metric_Pad1.05x0.95mm_HandSolder, F.Cu at (196.3, -31.8)
- added C133: 47nF, Capacitor_SMD:C_0603_1608Metric_Pad1.05x0.95mm_HandSolder, F.Cu at (183.2, -19.2)
- added C134: 4.7uF, Capacitor_SMD:C_0603_1608Metric_Pad1.05x0.95mm_HandSolder, F.Cu at (187.6, -24.2)
- added C135: 47nF, Capacitor_SMD:C_0603_1608Metric_Pad1.05x0.95mm_HandSolder, B.Cu at (275.2, 86.4)
- added C136: 47nF, Capacitor_SMD:C_0603_1608Metric_Pad1.05x0.95mm_HandSolder, F.Cu at (196.3, -29.2)
- added C137: 47nF, Capacitor_SMD:C_0603_1608Metric_Pad1.05x0.95mm_HandSolder, F.Cu at (187.6, -21.7)
- added C138: 0.47uF, Capacitor_SMD:C_0603_1608Metric_Pad1.05x0.95mm_HandSolder, F.Cu at (183.2, -16.7)
- added C139: 0.47uF, Capacitor_SMD:C_0603_1608Metric_Pad1.05x0.95mm_HandSolder, F.Cu at (200.6, -31.8)
- added C140: 0.47uF, Capacitor_SMD:C_0603_1608Metric_Pad1.05x0.95mm_HandSolder, B.Cu at (283.5, 88.0)
- added C141: 47nF, Capacitor_SMD:C_0603_1608Metric_Pad1.05x0.95mm_HandSolder, F.Cu at (191.9, -24.2)
- added C142: 47nF, Capacitor_SMD:C_0603_1608Metric_Pad1.05x0.95mm_HandSolder, F.Cu at (196.3, -26.7)
- added C143: 4.7uF, Capacitor_SMD:C_0603_1608Metric_Pad1.05x0.95mm_HandSolder, F.Cu at (200.6, -29.2)
- added C144: 4.7uF, Capacitor_SMD:C_0603_1608Metric_Pad1.05x0.95mm_HandSolder, F.Cu at (191.9, -21.7)
- added C145: 4.7uF, Capacitor_SMD:C_0603_1608Metric_Pad1.05x0.95mm_HandSolder, B.Cu at (283.5, 89.7)
- added C146: 47nF, Capacitor_SMD:C_0603_1608Metric_Pad1.05x0.95mm_HandSolder, F.Cu at (191.9, -19.2)
- added C147: 47nF, Capacitor_SMD:C_0603_1608Metric_Pad1.05x0.95mm_HandSolder, F.Cu at (196.3, -24.2)
- added C148: 47nF, Capacitor_SMD:C_0603_1608Metric_Pad1.05x0.95mm_HandSolder, F.Cu at (200.6, -26.7)
- added C149: 47nF, Capacitor_SMD:C_0603_1608Metric_Pad1.05x0.95mm_HandSolder, F.Cu at (196.3, -21.7)
- added C150: 0.47uF, Capacitor_SMD:C_0603_1608Metric_Pad1.05x0.95mm_HandSolder, F.Cu at (191.9, -16.7)
- added C151: 0.47uF, Capacitor_SMD:C_0603_1608Metric_Pad1.05x0.95mm_HandSolder, F.Cu at (196.3, -19.2)
- added C152: 4.7uF, Capacitor_SMD:C_0603_1608Metric_Pad1.05x0.95mm_HandSolder, F.Cu at (200.6, -24.2)
- C10, C23, C26, C29, C32, C35, C37, C41, C42, C6: moved to B.Cu
- C56, C60, C64, C65, C69, C72, C76, C82: value 100nF -> 10nF; moved to F.Cu
- C57, C61, C68: value 100nF -> 10nF
- C59, C63, C66, C67, C70, C71, C75, C81: value 4.7uF -> 10nF; moved to F.Cu
- C62, C74: value 4.7uF -> 10nF
- C73, C78: value 100nF -> 47nF; moved to F.Cu
- C77, C79, C83: value 4.7uF -> 47nF; moved to F.Cu
- C80: value 100nF -> 47nF
- moved C68 235.9 mm to (283.5, 84.7), turned to 0 degrees
- moved C80 223.2 mm to (290.1, 86.4), turned to 0 degrees
- moved U4 222.2 mm to (281.9, 71.1), turned to 90 degrees
- moved C79 220.7 mm to (187.6, -29.2), turned to 0 degrees
- moved CA1 220.0 mm to (242.8, 69.2), turned to 180 degrees
- moved C78 217.3 mm to (183.2, -26.7), turned to 0 degrees
- moved C66 213.9 mm to (178.9, -29.2), turned to 0 degrees
- moved C65 210.3 mm to (174.5, -26.7), turned to 0 degrees
- moved C62 210.2 mm to (290.1, 84.7)
- moved R20 208.7 mm to (246.2, 64.0), turned to 270 degrees
- moved C64 206.7 mm to (170.2, -24.2), turned to 0 degrees
- moved C71 206.4 mm to (178.9, -26.7), turned to 0 degrees
- moved C74 206.1 mm to (275.2, 84.7), turned to 180 degrees
- moved C67 205.3 mm to (170.2, -21.7), turned to 0 degrees
- moved C23 205.3 mm to (256.1, 67.2)
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- renumbered U1 to Ue1
Connections:
- net /FPGA/FPGA_JTDO renamed /FPGA_JTDO
- net /omega_2/BOOT_0 renamed /BOOT_0
- net /omega_2/OMG_JNRST renamed /OMG_JNRST
- net /omega_2/OMG_JTCK renamed /OMG_JTCK
- net /omega_2/OMG_JTDI renamed /OMG_JTDI
- net /omega_2/OMG_JTMS renamed /OMG_JTMS
- net /omega_2/OMG_JTRST renamed /OMG_JTRST
- net /proc/STM_JTDO renamed /STM_JTDO
- C61 pad 1: 1V2 FPGA -> 3V3 FPGA
- C62 pad 1: 1V2 FPGA -> 3V3 FPGA
- C63 pad 1: 3V3 FPGA -> 1V2 FPGA
- C65 pad 1: 1V2 FPGA -> 3V3 FPGA
- C66 pad 1: 1V2 FPGA -> 3V3 FPGA
- C70 pad 1: 1V2 FPGA -> 3V3 FPGA
- C73 pad 1: 1V2 FPGA -> 3V3 FPGA
- C74 pad 1: 1V2 FPGA -> 3V3 FPGA
- C75 pad 1: 3V3 FPGA -> 1V2 FPGA
- C81 pad 1: 3V3 FPGA -> 1V2 FPGA
- J2 pad 13: /omega_2/SDA_I2C -> I2C_SDA
- J2 pad 14: /omega_2/SCL_I2C -> I2C_SCL
- R3 pad 2: /proc/SPI1_MOSI -> SPI1_MOSI
- R4 pad 2: /omega_2/I2C1_SDA -> I2C_SCL
- R5 pad 2: /omega_2/I2C1_SCL -> I2C_SDA
- U2 pad 4: /omega_2/I2C1_SCL -> I2C_SDA
- U2 pad 5: /omega_2/I2C1_SDA -> I2C_SCL
- U3 pad 35: /proc/SPI1_SCK -> SPI1_SCK
- U4 pad 100: /proc/FMC_A20 -> FMC_A20
- U4 pad 101: /proc/FMC_A19 -> FMC_A19
- U4 pad 102: /proc/FMC_A23 -> FMC_A23
- U4 pad 112: /proc/FMC_NBL0 -> FMC_NBL0
- U4 pad 116: /proc/FMC_NL -> FMC_NL
- U4 pad 132: /proc/FMC_NWAIT -> FMC_NWAIT
- U4 pad 133: /proc/FMC_NWE -> FMC_NWE
- U4 pad 137: /proc/FMC_CLK -> FMC_CLK
- U4 pad 27: /proc/FMC_A18 -> FMC_A18
- U4 pad 29: /proc/FMC_A17 -> FMC_A17
- U4 pad 32: /proc/FMC_D15 -> FMC_D15
- U4 pad 41: /proc/FMC_D12 -> FMC_D12
- U4 pad 45: /proc/FMC_D9 -> FMC_D9
- U4 pad 46: /proc/FMC_D8 -> FMC_D8
- U4 pad 47: /proc/FMC_D7 -> FMC_D7
- U5 pad 114: /FPGA/FMC_D2 -> FMC_D2
- U5 pad 115: /FPGA/FMC_D3 -> FMC_D3
- U5 pad 118: /FPGA/FMC_NOE -> FMC_NOE
- U5 pad 123: /FPGA/FMC_NE1 -> FMC_NE1
- U5 pad 142: /FPGA/FMC_NBL1 -> FMC_NBL1
- U5 pad 4: /FPGA/FMC_A21 -> FMC_A21
- U5 pad 40: /rf_front_end/SPI1_CS_RF -> SPI1_CS_RF
- U5 pad 42: /rf_front_end/SPI1_MISO -> SPI1_MISO
- U5 pad 44: /rf_front_end/SPI1_CS_AD -> SPI1_CS_AD
- U5 pad 5: /FPGA/FMC_A22 -> FMC_A22
- U5 pad 58: /FPGA/FMC_D4 -> FMC_D4
- U5 pad 59: /FPGA/FMC_D5 -> FMC_D5
- U5 pad 60: /FPGA/FMC_D6 -> FMC_D6
- U5 pad 66: /FPGA/FMC_D10 -> FMC_D10
- U5 pad 67: /FPGA/FMC_D11 -> FMC_D11
- U5 pad 77: /FPGA/FMC_D13 -> FMC_D13
- U5 pad 78: /FPGA/FMC_D14 -> FMC_D14
- U5 pad 80: /FPGA/FMC_A16 -> FMC_A16
- U5 pad 85: /FPGA/FMC_D0 -> FMC_D0
- U5 pad 86: /FPGA/FMC_D1 -> FMC_D1
- U5 pad 89: /FPGA/FMC_A14 -> FMC_A14
- U5 pad 90: /FPGA/FMC_A15 -> FMC_A15
- Ue1 pad 18: /proc/SPI1_SCK -> SPI1_SCK
Routing:
- net 3V3 MCU: track 8.54 -> 4.74 mm

Commit message: organizacion PCB_V3
Parts:
- added C56: 4.7uF, Capacitor_SMD:C_0603_1608Metric_Pad1.05x0.95mm_HandSolder, B.Cu at (280.2, 86.5)
- added C57: 4.7uF, Capacitor_SMD:C_0603_1608Metric_Pad1.05x0.95mm_HandSolder, B.Cu at (281.7, 86.5)
- added C58: 4.7uF, Capacitor_SMD:C_0603_1608Metric_Pad1.05x0.95mm_HandSolder, B.Cu at (278.7, 86.5)
- added C59: 4.7uF, Capacitor_SMD:C_0603_1608Metric_Pad1.05x0.95mm_HandSolder, B.Cu at (273.2, 86.5)
- added C60: 4.7uF, Capacitor_SMD:C_0603_1608Metric_Pad1.05x0.95mm_HandSolder, B.Cu at (277.1, 86.5)
- added C61: 4.7uF, Capacitor_SMD:C_0603_1608Metric_Pad1.05x0.95mm_HandSolder, B.Cu at (298.8, 68.2)
- added C62: 4.7uF, Capacitor_SMD:C_0603_1608Metric_Pad1.05x0.95mm_HandSolder, B.Cu at (274.8, 55.2)
- added C63: 4.7uF, Capacitor_SMD:C_0603_1608Metric_Pad1.05x0.95mm_HandSolder, B.Cu at (266.1, 79.1)
- added C64: 4.7uF, Capacitor_SMD:C_0603_1608Metric_Pad1.05x0.95mm_HandSolder, B.Cu at (289.2, 86.4)
- added C65: 4.7uF, Capacitor_SMD:C_0603_1608Metric_Pad1.05x0.95mm_HandSolder, B.Cu at (266.1, 70.8)
- added C66: 4.7uF, Capacitor_SMD:C_0603_1608Metric_Pad1.05x0.95mm_HandSolder, B.Cu at (266.1, 72.4)
- added C67: 0.47uF, Capacitor_SMD:C_0603_1608Metric_Pad1.05x0.95mm_HandSolder, B.Cu at (298.8, 69.7)
- added C68: 0.47uF, Capacitor_SMD:C_0603_1608Metric_Pad1.05x0.95mm_HandSolder, B.Cu at (279.7, 55.3)
- added C69: 0.47uF, Capacitor_SMD:C_0603_1608Metric_Pad1.05x0.95mm_HandSolder, B.Cu at (266.1, 66.9)
- added C70: 0.47uF, Capacitor_SMD:C_0603_1608Metric_Pad1.05x0.95mm_HandSolder, B.Cu at (275.6, 86.5)
- added C71: 4.7uF, Capacitor_SMD:C_0603_1608Metric_Pad1.05x0.95mm_HandSolder, B.Cu at (266.1, 69.3)
- added C72: 4.7uF, Capacitor_SMD:C_0603_1608Metric_Pad1.05x0.95mm_HandSolder, B.Cu at (281.2, 55.3)
- added C73: 0.47uF, Capacitor_SMD:C_0603_1608Metric_Pad1.05x0.95mm_HandSolder, B.Cu at (298.8, 75.7)
- added C74: 0.47uF, Capacitor_SMD:C_0603_1608Metric_Pad1.05x0.95mm_HandSolder, B.Cu at (288.2, 55.3)
- added C75: 0.47uF, Capacitor_SMD:C_0603_1608Metric_Pad1.05x0.95mm_HandSolder, B.Cu at (266.1, 65.4)
- added C76: 0.47uF, Capacitor_SMD:C_0603_1608Metric_Pad1.05x0.95mm_HandSolder, B.Cu at (283.2, 86.5)
- added C77: 4.7uF, Capacitor_SMD:C_0603_1608Metric_Pad1.05x0.95mm_HandSolder, B.Cu at (282.7, 55.3)
- added C78: 0.47uF, Capacitor_SMD:C_0603_1608Metric_Pad1.05x0.95mm_HandSolder, B.Cu at (298.8, 71.2)
- added C79: 4.7uF, Capacitor_SMD:C_0603_1608Metric_Pad1.05x0.95mm_HandSolder, B.Cu at (298.8, 72.7)
- added C80: 0.47uF, Capacitor_SMD:C_0603_1608Metric_Pad1.05x0.95mm_HandSolder, B.Cu at (298.8, 74.2)
- C84, X2: moved to B.Cu
- moved X2 163.5 mm to (265.5, 75.7), turned to 90 degrees
- moved C84 155.8 mm to (262.4, 76.0), turned to 90 degrees
- moved C61 20.2 mm to (274.8, 97.4)
- moved C129 15.6 mm to (292.1, 99.4)
- moved C135 15.6 mm to (283.8, 99.4)
- moved C140 15.6 mm to (292.1, 101.0)
- moved C145 15.6 mm to (292.1, 102.7)
- moved C62 15.6 mm to (298.7, 97.7)
- moved C68 15.6 mm to (292.1, 97.7)
- moved C80 15.6 mm to (298.7, 99.4)
- moved C74 15.6 mm to (283.8, 97.7)
- renumbered Ue1 to U1
Connections:
- net /BOOT_0 renamed /omega_2/BOOT_0
- net /FPGA_JTDO renamed /FPGA/FPGA_JTDO
- net /OMG_JNRST renamed /omega_2/OMG_JNRST
- net /OMG_JTCK renamed /omega_2/OMG_JTCK
- net /OMG_JTDI renamed /omega_2/OMG_JTDI
- net /OMG_JTMS renamed /omega_2/OMG_JTMS
- net /OMG_JTRST renamed /omega_2/OMG_JTRST
- net /STM_JTDO renamed /proc/STM_JTDO
- J2 pad 13: I2C_SDA -> /omega_2/SDA_I2C
- J2 pad 14: I2C_SCL -> /omega_2/SCL_I2C
- R4 pad 2: I2C_SCL -> /omega_2/I2C1_SDA
- R5 pad 2: I2C_SDA -> /omega_2/I2C1_SCL
- U2 pad 4: I2C_SDA -> /omega_2/I2C1_SCL
- U2 pad 5: I2C_SCL -> /omega_2/I2C1_SDA
- U3 pad 36: SPI1_CS_AD -> /proc/SPI1_CS_AD
- U4 pad 111: FMC_NBL1 -> /proc/FMC_NBL1
- U4 pad 112: FMC_NBL0 -> /proc/FMC_NBL0
- U4 pad 132: FMC_NWAIT -> /proc/FMC_NWAIT
- U4 pad 133: FMC_NWE -> /proc/FMC_NWE
- U4 pad 137: FMC_CLK -> /proc/FMC_CLK
- U4 pad 30: FMC_A16 -> /proc/FMC_A16
- U5 pad 1: FMC_A23 -> /FPGA/FMC_A23
- U5 pad 114: FMC_D2 -> /FPGA/FMC_D2
- U5 pad 115: FMC_D3 -> /FPGA/FMC_D3
- U5 pad 118: FMC_NOE -> /FPGA/FMC_NOE
- U5 pad 123: FMC_NE1 -> /FPGA/FMC_NE1
- U5 pad 137: FMC_NL -> /FPGA/FMC_NL
- U5 pad 2: FMC_A19 -> /FPGA/FMC_A19
- U5 pad 3: FMC_A20 -> /FPGA/FMC_A20
- U5 pad 4: FMC_A21 -> /FPGA/FMC_A21
- U5 pad 40: SPI1_CS_RF -> /rf_front_end/SPI1_CS_RF
- U5 pad 41: SPI1_SCK -> /rf_front_end/SPI1_SCK
- U5 pad 42: SPI1_MISO -> /rf_front_end/SPI1_MISO
- U5 pad 43: SPI1_MOSI -> /rf_front_end/SPI1_MOSI
- U5 pad 5: FMC_A22 -> /FPGA/FMC_A22
- U5 pad 58: FMC_D4 -> /FPGA/FMC_D4
- U5 pad 59: FMC_D5 -> /FPGA/FMC_D5
- U5 pad 60: FMC_D6 -> /FPGA/FMC_D6
- U5 pad 63: FMC_D7 -> /FPGA/FMC_D7
- U5 pad 64: FMC_D8 -> /FPGA/FMC_D8
- U5 pad 65: FMC_D9 -> /FPGA/FMC_D9
- U5 pad 66: FMC_D10 -> /FPGA/FMC_D10
- U5 pad 67: FMC_D11 -> /FPGA/FMC_D11
- U5 pad 68: FMC_D12 -> /FPGA/FMC_D12
- U5 pad 77: FMC_D13 -> /FPGA/FMC_D13
- U5 pad 78: FMC_D14 -> /FPGA/FMC_D14
- U5 pad 79: FMC_D15 -> /FPGA/FMC_D15
- U5 pad 81: FMC_A17 -> /FPGA/FMC_A17
- U5 pad 82: FMC_A18 -> /FPGA/FMC_A18
- U5 pad 85: FMC_D0 -> /FPGA/FMC_D0
- U5 pad 86: FMC_D1 -> /FPGA/FMC_D1
- U5 pad 89: FMC_A14 -> /FPGA/FMC_A14
- U5 pad 90: FMC_A15 -> /FPGA/FMC_A15
