File: HW/shield_SDR_UN/shield_SDR_UN.kicad_pcb (KiCad board)
At the start: 2 copper layers, 100 x 100 mm, 294 parts, among them J1 Conn_02x09_Odd_Even, J2 Conn_02x08_Odd_Even, J3 Conn_02x10_Top_Bottom, J4 USB_B_Micro, J5 USB_A, J6 Conn_02x06_Odd_Even, P1 GSG-RF-CONN, P2 GSG-RF-CONN, Q1 MOSFET_P, T1 BALUN, T2 BALUN, U1 MAX2830, U2 SI5351C, U3 MAX5864, U4 XC6SLX9-2TQG144C, U5 STM32F722ZET, U6 ZLDO1117G33TA, U7 ZLDO1117G33TA, U8 ZLDO1117G12TA, U9 OMEGA_2, X1 GSG-XTAL4PIN, X2 ASE-xxxMHz, X3 CRYSTAL, X4 GSG-XTAL4PIN

Commit message: Capacitors of RF front-end edited, components placed in the PCB
Parts:
- removed C127, C129, C130, C131, C132, C133, C135, C136, C137, C141, C142, C146, C147, C148, C149, C83: 47nF, Capacitor_SMD:C_0603_1608Metric_Pad1.05x0.95mm_HandSolder
- removed C128, C138, C139, C140, C150, C151: 0.47uF, Capacitor_SMD:C_0603_1608Metric_Pad1.05x0.95mm_HandSolder
- removed C134, C143, C144, C145, C152: 4.7uF, Capacitor_SMD:C_0603_1608Metric_Pad1.05x0.95mm_HandSolder
- removed C18, C23, C24, C25, C29, C30, C31, C35, C36, C41: 2.2uF, Capacitor_SMD:C_0603_1608Metric_Pad1.05x0.95mm_HandSolder
- removed C26, C27, C28, C32, C33, C34, C37, C38, C42: 100nF, Capacitor_SMD:C_0603_1608Metric_Pad1.05x0.95mm_HandSolder
- removed the C56 at (170.2, -31.8)
- removed the C57 at (89.4, 141.0)
- removed the C58 at (89.4, 139.5)
- removed the C59 at (170.2, -29.2)
- removed the C60 at (174.5, -31.8)
- removed the C61 at (274.8, 97.4)
- removed the C62 at (298.7, 97.7)
- removed the C63 at (178.9, -31.8)
- removed the C64 at (170.2, -24.2)
- removed the C65 at (174.5, -26.7)
- removed the C66 at (178.9, -29.2)
- removed the C67 at (170.2, -21.7)
- removed the C68 at (292.1, 97.7)
- removed the C69 at (170.2, -19.2)
- removed the C70 at (174.5, -24.2)
- removed the C71 at (178.9, -26.7)
- removed the C72 at (183.2, -29.2)
- removed the C73 at (174.5, -21.7)
- removed the C74 at (283.8, 97.7)
- removed the C75 at (187.6, -31.8)
- removed the C76 at (174.5, -19.2)
- removed the C77 at (178.9, -24.2)
- removed the C78 at (183.2, -26.7)
- removed the C79 at (187.6, -29.2)
- removed the C80 at (298.7, 99.4)
- removed C81, C82: 10nF, Capacitor_SMD:C_0603_1608Metric_Pad1.05x0.95mm_HandSolder
- C12, C3: value 2.2uF -> 100p; moved to B.Cu
- C13, C19: value 2.2uF -> 10n; moved to B.Cu
- C15, C16, C21: value 100nF -> 10n; moved to B.Cu
- C22, C8, C9: value 100nF -> 100p; moved to B.Cu
- C39, C40: footprint Capacitor_SMD:C_0603_1608Metric_Pad1.05x0.95mm_HandSolder -> Capacitor_SMD:C_0402_1005Metric
- C4: value 2.2uF -> 10u; moved to B.Cu
- C48, CA1, CA2, CA3: moved to B.Cu
- C5: footprint Capacitor_SMD:C_0805_2012Metric_Pad1.15x1.40mm_HandSolder -> Capacitor_SMD:C_0603_1608Metric_Pad1.05x0.95mm_HandSolder
- moved C44 212.6 mm to (241.3, 72.9), turned to 90 degrees
- moved C4 212.3 mm to (230.9, 63.7), turned to 180 degrees
- moved C48 208.7 mm to (244.1, 65.8), turned to 180 degrees
- moved R22 208.3 mm to (256.4, 80.0), turned to 180 degrees
- moved R8 208.2 mm to (245.2, 72.0), turned to 180 degrees
- moved C40 207.6 mm to (231.6, 68.2)
- moved T2 206.0 mm to (229.0, 67.7), turned to 90 degrees
- moved C3 205.8 mm to (230.9, 62.2), turned to 180 degrees
- moved C9 205.4 mm to (235.1, 72.7), turned to 270 degrees
- moved R23 202.4 mm to (256.4, 81.7), turned to 180 degrees
- moved R21 201.7 mm to (256.4, 83.2)
- moved C43 201.6 mm to (242.2, 78.4), turned to 180 degrees
- moved P2 201.1 mm to (222.3, 73.3), turned to 270 degrees
- moved C49 200.8 mm to (249.9, 75.5), turned to 90 degrees
- moved P1 199.5 mm to (222.3, 62.0), turned to 270 degrees
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Connections:
- net /FPGA/FPGA_JTDO renamed /FPGA_JTDO
- net /omega_2/BOOT_0 renamed /BOOT_0
- net /omega_2/OMG_JNRST renamed /OMG_JNRST
- net /omega_2/OMG_JTCK renamed /OMG_JTCK
- net /omega_2/OMG_JTDI renamed /OMG_JTDI
- net /omega_2/OMG_JTMS renamed /OMG_JTMS
- net /omega_2/OMG_JTRST renamed /OMG_JTRST
- net /proc/STM_JTDO renamed /STM_JTDO
- J2 pad 13: /omega_2/SDA_I2C -> I2C_SDA
- J2 pad 14: /omega_2/SCL_I2C -> I2C_SCL
- R4 pad 2: /omega_2/I2C1_SDA -> I2C_SCL
- R5 pad 2: /omega_2/I2C1_SCL -> I2C_SDA
- U2 pad 4: /omega_2/I2C1_SCL -> I2C_SDA
- U2 pad 5: /omega_2/I2C1_SDA -> I2C_SCL
- U3 pad 36: /proc/SPI1_CS_AD -> SPI1_CS_AD
- U4 pad 111: /proc/FMC_NBL1 -> FMC_NBL1
- U4 pad 112: /proc/FMC_NBL0 -> FMC_NBL0
- U4 pad 132: /proc/FMC_NWAIT -> FMC_NWAIT
- U4 pad 133: /proc/FMC_NWE -> FMC_NWE
- U4 pad 137: /proc/FMC_CLK -> FMC_CLK
- U4 pad 30: /proc/FMC_A16 -> FMC_A16
- U5 pad 1: /FPGA/FMC_A23 -> FMC_A23
- U5 pad 114: /FPGA/FMC_D2 -> FMC_D2
- U5 pad 115: /FPGA/FMC_D3 -> FMC_D3
- U5 pad 118: /FPGA/FMC_NOE -> FMC_NOE
- U5 pad 123: /FPGA/FMC_NE1 -> FMC_NE1
- U5 pad 137: /FPGA/FMC_NL -> FMC_NL
- U5 pad 2: /FPGA/FMC_A19 -> FMC_A19
- U5 pad 3: /FPGA/FMC_A20 -> FMC_A20
- U5 pad 4: /FPGA/FMC_A21 -> FMC_A21
- U5 pad 40: /rf_front_end/SPI1_CS_RF -> SPI1_CS_RF
- U5 pad 41: /rf_front_end/SPI1_SCK -> SPI1_SCK
- U5 pad 42: /rf_front_end/SPI1_MISO -> SPI1_MISO
- U5 pad 43: /rf_front_end/SPI1_MOSI -> SPI1_MOSI
- U5 pad 5: /FPGA/FMC_A22 -> FMC_A22
- U5 pad 58: /FPGA/FMC_D4 -> FMC_D4
- U5 pad 59: /FPGA/FMC_D5 -> FMC_D5
- U5 pad 60: /FPGA/FMC_D6 -> FMC_D6
- U5 pad 63: /FPGA/FMC_D7 -> FMC_D7
- U5 pad 64: /FPGA/FMC_D8 -> FMC_D8
- U5 pad 65: /FPGA/FMC_D9 -> FMC_D9
- U5 pad 66: /FPGA/FMC_D10 -> FMC_D10
- U5 pad 67: /FPGA/FMC_D11 -> FMC_D11
- U5 pad 68: /FPGA/FMC_D12 -> FMC_D12
- U5 pad 77: /FPGA/FMC_D13 -> FMC_D13
- U5 pad 78: /FPGA/FMC_D14 -> FMC_D14
- U5 pad 79: /FPGA/FMC_D15 -> FMC_D15
- U5 pad 81: /FPGA/FMC_A17 -> FMC_A17
- U5 pad 82: /FPGA/FMC_A18 -> FMC_A18
- U5 pad 85: /FPGA/FMC_D0 -> FMC_D0
- U5 pad 86: /FPGA/FMC_D1 -> FMC_D1
- U5 pad 89: /FPGA/FMC_A14 -> FMC_A14
- U5 pad 90: /FPGA/FMC_A15 -> FMC_A15

Commit message: organizacion PCB_V4
Parts:
- moved J1 361.8 mm to (379.8, 126.6), turned to 180 degrees
- moved R43 333.9 mm to (370.6, 70.4), turned to 180 degrees
- moved R47 316.8 mm to (370.6, 72.0)
- moved R38 312.0 mm to (371.5, 109.8)
- moved R24 303.1 mm to (371.4, 126.3)
- moved R29 301.6 mm to (371.5, 111.3), turned to 180 degrees
- moved R28 301.4 mm to (371.5, 114.3), turned to 180 degrees
- moved J2 275.4 mm to (379.9, 83.7), turned to 180 degrees
- moved R46 265.1 mm to (370.6, 75.0)
- moved R40 256.4 mm to (370.6, 79.5), turned to 180 degrees
- moved R30 253.5 mm to (371.5, 108.3), turned to 180 degrees
- moved R42 252.9 mm to (370.6, 73.5), turned to 180 degrees
- moved R27 252.5 mm to (371.5, 117.3), turned to 180 degrees
- moved R45 252.0 mm to (370.6, 77.9)
- moved R36 250.6 mm to (371.5, 115.8)
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Connections:
- net /BOOT_0 renamed /omega_2/BOOT_0
- net /FPGA_JTDO renamed /FPGA/FPGA_JTDO
- net /OMG_JNRST renamed /omega_2/OMG_JNRST
- net /OMG_JTCK renamed /omega_2/OMG_JTCK
- net /OMG_JTDI renamed /omega_2/OMG_JTDI
- net /OMG_JTMS renamed /omega_2/OMG_JTMS
- net /OMG_JTRST renamed /omega_2/OMG_JTRST
- net /STM_JTDO renamed /proc/STM_JTDO
- J2 pad 13: I2C_SDA -> /omega_2/SDA_I2C
- J2 pad 14: I2C_SCL -> /omega_2/SCL_I2C
- R4 pad 2: I2C_SCL -> /omega_2/I2C1_SDA
- R5 pad 2: I2C_SDA -> /omega_2/I2C1_SCL
- U2 pad 4: I2C_SDA -> /omega_2/I2C1_SCL
- U2 pad 5: I2C_SCL -> /omega_2/I2C1_SDA
- U3 pad 36: SPI1_CS_AD -> /proc/SPI1_CS_AD
- U4 pad 139: FMC_D2 -> /proc/FMC_D2
- U4 pad 56: adDD9 -> adDA0
- U4 pad 57: adDD8 -> adDA1
- U4 pad 58: adDD7 -> adDA2
- U4 pad 59: adDD6 -> adDA3
- U4 pad 60: adDD5 -> adDA4
- U4 pad 61: adDD4 -> adDA5
- U4 pad 62: adDD3 -> adDA6
- U4 pad 64: adDD2 -> adDA7
- U4 pad 65: adDD1 -> adDD0
- U4 pad 66: adDD0 -> adDD1
- U4 pad 67: adDA7 -> adDD2
- U4 pad 69: adDA6 -> adDD3
- U4 pad 70: adDA5 -> adDD4
- U4 pad 74: adDA4 -> adDD5
- U4 pad 75: adDA3 -> adDD6
- U4 pad 78: adDA2 -> adDD7
- U4 pad 79: adDA1 -> adDD8
- U4 pad 80: adDA0 -> adDD9
- U5 pad 1: FMC_A23 -> /FPGA/FMC_A23
- U5 pad 115: FMC_D3 -> /FPGA/FMC_D3
- U5 pad 117: FMC_CLK -> /FPGA/FMC_CLK
- U5 pad 118: FMC_NOE -> /FPGA/FMC_NOE
- U5 pad 119: FMC_NWE -> /FPGA/FMC_NWE
- U5 pad 122: FMC_NWAIT -> /FPGA/FMC_NWAIT
- U5 pad 123: FMC_NE1 -> /FPGA/FMC_NE1
- U5 pad 137: FMC_NL -> /FPGA/FMC_NL
- U5 pad 141: FMC_NBL0 -> /FPGA/FMC_NBL0
- U5 pad 142: FMC_NBL1 -> /FPGA/FMC_NBL1
- U5 pad 2: FMC_A19 -> /FPGA/FMC_A19
- U5 pad 3: FMC_A20 -> /FPGA/FMC_A20
- U5 pad 4: FMC_A21 -> /FPGA/FMC_A21
- U5 pad 40: SPI1_CS_RF -> /rf_front_end/SPI1_CS_RF
- U5 pad 41: SPI1_SCK -> /rf_front_end/SPI1_SCK
- U5 pad 42: SPI1_MISO -> /rf_front_end/SPI1_MISO
- U5 pad 43: SPI1_MOSI -> /rf_front_end/SPI1_MOSI
- U5 pad 5: FMC_A22 -> /FPGA/FMC_A22
- U5 pad 58: FMC_D4 -> /FPGA/FMC_D4
- U5 pad 59: FMC_D5 -> /FPGA/FMC_D5
- U5 pad 60: FMC_D6 -> /FPGA/FMC_D6
- U5 pad 63: FMC_D7 -> /FPGA/FMC_D7
- U5 pad 64: FMC_D8 -> /FPGA/FMC_D8
- U5 pad 65: FMC_D9 -> /FPGA/FMC_D9
- U5 pad 66: FMC_D10 -> /FPGA/FMC_D10
- U5 pad 67: FMC_D11 -> /FPGA/FMC_D11
- U5 pad 68: FMC_D12 -> /FPGA/FMC_D12
- U5 pad 77: FMC_D13 -> /FPGA/FMC_D13
- U5 pad 78: FMC_D14 -> /FPGA/FMC_D14
- U5 pad 79: FMC_D15 -> /FPGA/FMC_D15
- U5 pad 80: FMC_A16 -> /FPGA/FMC_A16
- U5 pad 81: FMC_A17 -> /FPGA/FMC_A17
- U5 pad 82: FMC_A18 -> /FPGA/FMC_A18
- U5 pad 85: FMC_D0 -> /FPGA/FMC_D0
- U5 pad 86: FMC_D1 -> /FPGA/FMC_D1
- U5 pad 89: FMC_A14 -> /FPGA/FMC_A14
- U5 pad 90: FMC_A15 -> /FPGA/FMC_A15

Commit message: PCB :)
Parts:
- BT1, C124, C125, D10, D11: moved to B.Cu
- moved BT1 43.6 mm to (303.0, 56.9)
- moved J2 40.6 mm to (341.7, 97.2)
- moved R41 39.9 mm to (333.9, 92.1)
- moved R45 39.9 mm to (333.9, 93.6)
- moved R40 39.9 mm to (333.9, 95.1)
- moved R42 39.9 mm to (333.9, 89.1)
- moved R46 39.9 mm to (333.9, 90.6)
- moved R43 39.9 mm to (333.9, 86.1)
- moved R44 39.9 mm to (333.9, 96.6)
- moved R47 39.9 mm to (333.9, 87.6)
- moved R48 39.9 mm to (333.9, 84.5)
- moved J1 38.0 mm to (341.8, 125.2)
- moved R25 38.0 mm to (333.4, 121.9)
- moved R30 38.0 mm to (333.5, 106.8)
- moved R33 38.0 mm to (333.4, 123.4)
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
Commit message: PCB route V1
Parts:
- removed C86: 100nF, Capacitor_SMD:C_0603_1608Metric_Pad1.05x0.95mm_HandSolder
- added C18: 100nF, Capacitor_SMD:C_0603_1608Metric_Pad1.05x0.95mm_HandSolder, F.Cu at (314.5, 70.4)
- C11, C114, C115, C117, C118, C119, C121, C14, C17, C20, C51, C52, C53, C54, L3, R24, R25, R26, R27, R28, R29, R30, R33, R34, R35, R36, R37, R38, R39, R40, R41, R42, R43, R44, R45, R46, R47, R48, R58, U7, U8: moved to B.Cu
- D7: footprint LED_SMD:LED_0603_1608Metric_Pad1.05x0.95mm_HandSolder -> LED_SMD:LED_0805_2012Metric_Pad1.15x1.40mm_HandSolder
- moved S1 292.6 mm to (318.7, 62.7), turned to 90 degrees
- moved D2 271.4 mm to (298.6, 70.2), turned to 270 degrees
- moved C85 270.6 mm to (312.6, 60.9), turned to 270 degrees
- moved D3 254.3 mm to (296.4, 70.2), turned to 270 degrees
- moved S2 251.4 mm to (318.7, 72.2), turned to 90 degrees
- moved D4 240.3 mm to (264.6, 80.9)
- moved R51 211.2 mm to (268.4, 79.6)
- moved R50 210.7 mm to (312.9, 70.4), turned to 270 degrees
- moved R49 204.8 mm to (314.2, 60.9), turned to 270 degrees
- moved R32 183.6 mm to (296.3, 74.2), turned to 90 degrees
- moved R31 180.6 mm to (298.6, 74.2), turned to 90 degrees
- moved S3 179.9 mm to (221.2, 97.8), turned to 270 degrees
- moved R53 164.9 mm to (268.5, 101.5)
- moved R52 159.8 mm to (268.4, 81.3), turned to 180 degrees
- moved C116 146.4 mm to (313.3, 139.0), turned to 180 degrees
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Connections:
- J2 pad 13: /omega_2/SDA_I2C -> I2C_SDA
- J2 pad 14: /omega_2/SCL_I2C -> I2C_SCL
- J6 pad 1: /omega_2/3V3_OMEG -> 3V3 MCU
- J6 pad 2: /omega_2/3V3_OMEG -> 3V3 MCU
- R35 pad 1: /FPGA/FPGA_GPIO_01 -> /FPGA/FPGA_GPIO_04
- R49 pad 1: 3V3 FPGA -> /FPGA/BTN1
- R49 pad 2: /FPGA/BTN1 -> GND
- R50 pad 1: 3V3 FPGA -> /FPGA/BTN2
- R50 pad 2: /FPGA/BTN2 -> GND
- S1 pad 3: GND -> 3V3 FPGA
- S1 pad 4: GND -> 3V3 FPGA
- S2 pad 3: GND -> 3V3 FPGA
- S2 pad 4: GND -> 3V3 FPGA
- U3 pad 36: /proc/SPI1_CS_AD -> SPI1_CS_AD
- U4 pad 112: FMC_NBL0 -> /proc/FMC_NBL0
- U4 pad 132: FMC_NWAIT -> /proc/FMC_NWAIT
- U4 pad 133: FMC_NWE -> /proc/FMC_NWE
- U4 pad 139: /proc/FMC_D2 -> FMC_D2
- U4 pad 44: FMC_D10 -> /proc/FMC_D10
- U5 pad 114: FMC_D2 -> /FPGA/FMC_D2
- U5 pad 119: /FPGA/FMC_NWE -> FMC_NWE
- U5 pad 122: /FPGA/FMC_NWAIT -> FMC_NWAIT
- U5 pad 141: /FPGA/FMC_NBL0 -> FMC_NBL0
- U5 pad 44: SPI1_CS_AD -> /rf_front_end/SPI1_CS_AD
- U5 pad 66: /FPGA/FMC_D10 -> FMC_D10
Routing:
- net /omega_2/O_SPI_MOSI: track 0.00 -> 61.7 mm
- net /omega_2/O_SPI_MISO: track 0.00 -> 60.6 mm
- net /omega_2/O_SPI_CS1: track 0.00 -> 57.9 mm
- net /omega_2/O_SPI_CLK: track 0.00 -> 56.7 mm
- net /omega_2/SER_RX0: track 0.00 -> 38.3 mm
- net /omega_2/SER_TX0: track 0.00 -> 33.4 mm
- net /FPGA/FPGA_GPIO_04: track 0.00 -> 28.3 mm, vias 0 -> 2
- net /FPGA/FPGA_GPIO_05: track 0.00 -> 26.6 mm, vias 0 -> 2
- net /FPGA/FPGA_GPIO_06: track 0.00 -> 24.4 mm, vias 0 -> 2
- net I2C_SDA: track 0.00 -> 24.0 mm
- net /FPGA/FPGA_GPIO_07: track 0.00 -> 21.9 mm, vias 0 -> 2
- net /FPGA/FPGA_GPIO_08: track 0.00 -> 20.6 mm, vias 0 -> 2
- net I2C_SCL: track 0.00 -> 20.6 mm
- net /FPGA/FPGA_GPIO_09: track 0.00 -> 19.5 mm, vias 0 -> 2
- net /FPGA/FPGA_GPIO_10: track 0.00 -> 18.3 mm, vias 0 -> 2
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Other:
- net class Power added: clearance 0.16, trace_width 0.9, via_dia 0.8, via_drill 0.4
- rule trace_min: 0.2 -> 0.16
- board text added: "Camargo vea esta belleza, pongame 5"
